File: RAMPS-FD/Extra_Mosfets.sch (KiCad schematic (older format))
At the start: 12 parts, among them P901 D12, P902 D2, Q901 DMN2075U, Q902 DMN2075U

Commit message: Inital Commit RAMPS FD v2.3. SPI Support for every Driver added.
Parts:
- D901, D902: symbol LED-RESCUE-RAMPS-FD -> RAMPS-FD-rescue:LED-RESCUE-RAMPS-FD
- D903, D904: symbol D -> RAMPS-FD-rescue:D
- P901, P902: symbol CONN_2 -> RAMPS-FD-rescue:CONN_2
- Q901, Q902: symbol MOSFET_N -> RMC:MOSFET_N
- R901, R902, R905, R906: symbol R -> RAMPS-FD-rescue:R
Changed lines of the file:
@@
-EESchema Schematic File Version 2
-LIBS:RAMPS-FD-rescue
-LIBS:power
-LIBS:device
-LIBS:transistors
-LIBS:conn
-LIBS:linear
-LIBS:regul
-LIBS:74xx
-LIBS:cmos4000
-LIBS:adc-dac
-LIBS:memory
-LIBS:xilinx
-LIBS:microcontrollers
-LIBS:dsp
-LIBS:microchip
-LIBS:analog_switches
-LIBS:motorola
-LIBS:texas
-LIBS:intel
-LIBS:audio
-LIBS:interface
-LIBS:digital-audio
-LIBS:philips
-LIBS:display
-LIBS:cypress
-LIBS:siliconi
-LIBS:opto
-LIBS:atmel
-LIBS:contrib
-LIBS:valves
-LIBS:RMC
-LIBS:RAMPS-FD-cache
-EELAYER 25 0
+EESchema Schematic File Version 4
+EELAYER 30 0
 EELAYER END
 $Descr A4 11693 8268
@@
 Sheet 9 10
 Title "RAMPS-FD (RAMPS for Arduino Due)"
-Date "2016-07-17"
-Rev "v2.2"
+Date "2019-04-13"
+Rev "v2.3"
 Comp ""
-Comment1 "Derived from RAMPS 1.4 reprap.org/wiki/RAMPS1.4"
+Comment1 "Derived from RAMPS FD 2.2 by Bob Cousins github.com/bobc/bobc_hardware/"
 Comment2 "GPL v3"
-Comment3 "Bob Cousins 2016"
+Comment3 "Marius Krause 2019"
 Comment4 ""
 $EndDescr
@@
 	3500 850  3500 1350
 $Comp
-L MOSFET_N Q901
+L RMC:MOSFET_N Q901
 U 1 1 523E5FE5
 P 3425 2475
@@
 $EndComp
 $Comp
-L GNDPWR #PWR0110
+L RAMPS-FD-rescue:GNDPWR #PWR0110
 U 1 1 523E5FF8
 P 3500 3350
@@
 $EndComp
 $Comp
-L CONN_2 P901
+L RAMPS-FD-rescue:CONN_2 P901
 U 1 1 523E5FFE
 P 4850 1950
@@
 $EndComp
 $Comp
-L D D903
+L RAMPS-FD-rescue:D D903
 U 1 1 523E6004
 P 3500 1500
@@
 $EndComp
 $Comp
-L LED-RESCUE-RAMPS-FD D901
+L RAMPS-FD-rescue:LED-RESCUE-RAMPS-FD D901
 U 1 1 523E6017
 P 3000 1800
@@
 $EndComp
 $Comp
-L R R905
+L RAMPS-FD-rescue:R R905
 U 1 1 523E601D
 P 3000 1300
@@
 FET5_BUF
 $Comp
-L +12P #PWR0111
+L power:+12P #PWR0111
 U 1 1 523E6026
 P 3500 850
@@
 	3500 4050 3500 4550
 $Comp
-L MOSFET_N Q902
+L RMC:MOSFET_N Q902
 U 1 1 523E66A5
 P 3425 5675
@@
 $EndComp
 $Comp
-L GNDPWR #PWR0112
+L RAMPS-FD-rescue:GNDPWR #PWR0112
 U 1 1 523E66AB
 P 3500 6325
@@
 $EndComp
 $Comp
-L CONN_2 P902
+L RAMPS-FD-rescue:CONN_2 P902
 U 1 1 523E66B1
 P 4850 5150
@@
 $EndComp
 $Comp
-L D D904
+L RAMPS-FD-rescue:D D904
 U 1 1 523E66B7
 P 3500 4700
@@
 $EndComp
 $Comp
-L LED-RESCUE-RAMPS-FD D902
+L RAMPS-FD-rescue:LED-RESCUE-RAMPS-FD D902
 U 1 1 523E66BD
 P 3000 5000
@@
 $EndComp
 $Comp
-L R R906
+L RAMPS-FD-rescue:R R906
 U 1 1 523E66C3
 P 3000 4500
@@
 FET6_BUF
 $Comp
-L +12P #PWR0113
+L power:+12P #PWR0113
 U 1 1 523E66CA
 P 3500 4050
@@
 P_FET6
 $Comp
-L R R902
+L RAMPS-FD-rescue:R R902
 U 1 1 52C42B15
 P 2300 2550
@@
 	2450 2550 3125 2550
 $Comp
-L R R901
+L RAMPS-FD-rescue:R R901
 U 1 1 52C42B98
 P 2325 5750

Commit message: Added UART for Communication with TMC2209 Drivers, improved inverse-polarity protection, added Driver Protection. Two Layer Design
Parts:
- D28: renamed from D903; value ES1F -> 2CZ4007; footprint rmc:DO-214AC -> RAMPS-FD:D_SOD-123F; symbol RAMPS-FD-rescue:D -> RAMPS-FD:2CZ4007; Fitted (none) -> yes; Ordering (none) -> LCSC: C85712; Price (USD) (none) -> 0,05; Rating (none) -> #1kV #1A
- D29: renamed from D901; value LED RED -> LED_0603_RED; footprint rmc:LED-0805_RED -> RAMPS-FD:LED_0603; symbol RAMPS-FD-rescue:LED-RESCUE-RAMPS-FD -> RAMPS-FD:LED_0603_RED; Fitted (none) -> yes; Ordering (none) -> LCSC: C192315; Price (USD) (none) -> 0,018284
- D30: renamed from D904; value ES1F -> 2CZ4007; footprint rmc:DO-214AC -> RAMPS-FD:D_SOD-123F; symbol RAMPS-FD-rescue:D -> RAMPS-FD:2CZ4007; Fitted (none) -> yes; Ordering (none) -> LCSC: C85712; Price (USD) (none) -> 0,05; Rating (none) -> #1kV #1A
- D31: renamed from D902; value LED RED -> LED_0603_RED; footprint rmc:LED-0805_RED -> RAMPS-FD:LED_0603; symbol RAMPS-FD-rescue:LED-RESCUE-RAMPS-FD -> RAMPS-FD:LED_0603_RED; Fitted (none) -> yes; Ordering (none) -> LCSC: C192315; Price (USD) (none) -> 0,018284
- J30: renamed from P901; value D12 -> 2x1PinHeader; footprint rmc:CONN_KK_2.54_2W -> RAMPS-FD:PinHeader_1x02_P2.54mm_Vertical; symbol RAMPS-FD-rescue:CONN_2 -> RAMPS-FD:2x1PinHeader; Fitted (none) -> yes; Ordering (none) -> LCSC: C124375; Price (USD) (none) -> 0,015147
- J31: renamed from P902; value D2 -> 2x1PinHeader; footprint rmc:CONN_KK_2.54_2W -> RAMPS-FD:PinHeader_1x02_P2.54mm_Vertical; symbol RAMPS-FD-rescue:CONN_2 -> RAMPS-FD:2x1PinHeader; Fitted (none) -> yes; Ordering (none) -> LCSC: C124375; Price (USD) (none) -> 0,015147
- Q10: renamed from Q901; value DMN2075U -> NCE3416; footprint libcms:SOT23GDS -> RAMPS-FD:SOT-23; symbol RMC:MOSFET_N -> RAMPS-FD:NCE3416; Fitted (none) -> yes; Ordering (none) -> LCSC: C113491; Price (USD) (none) -> 0,033091; Rating (none) -> #20V #6.5A
- Q11: renamed from Q902; value DMN2075U -> NCE3416; footprint libcms:SOT23GDS -> RAMPS-FD:SOT-23; symbol RMC:MOSFET_N -> RAMPS-FD:NCE3416; Fitted (none) -> yes; Ordering (none) -> LCSC: C113491; Price (USD) (none) -> 0,033091; Rating (none) -> #20V #6.5A
- R34: renamed from R905; footprint Resistors_SMD:R_0603 -> RAMPS-FD:R_0603; symbol RAMPS-FD-rescue:R -> RAMPS-FD:1k; Fitted (none) -> yes; Ordering (none) -> LCSC: C328340; Price (USD) (none) -> 0,003087
- R35: renamed from R902; value 220R -> 33R; footprint Resistors_SMD:R_0603 -> RAMPS-FD:R_0603; symbol RAMPS-FD-rescue:R -> RAMPS-FD:33R; Fitted (none) -> yes; Ordering (none) -> LCSC: C325638; Price (USD) (none) -> 0,002066
- R36: renamed from R906; footprint Resistors_SMD:R_0603 -> RAMPS-FD:R_0603; symbol RAMPS-FD-rescue:R -> RAMPS-FD:1k; Fitted (none) -> yes; Ordering (none) -> LCSC: C328340; Price (USD) (none) -> 0,003087
- R37: renamed from R901; value 220R -> 33R; footprint Resistors_SMD:R_0603 -> RAMPS-FD:R_0603; symbol RAMPS-FD-rescue:R -> RAMPS-FD:33R; Fitted (none) -> yes; Ordering (none) -> LCSC: C325638; Price (USD) (none) -> 0,002066
Connections:
- wire segments 24 -> 37
