File: RAMPS-FD/Power.sch (KiCad schematic (older format))
At the start: 21 parts, among them J1 NET-TIE, P101 HB_IN, P105 12V-AUX, P108 POWER_IN, P219 EXT_5V, U3 R-78E12-0.5, U4 L7805CV-DG

Commit message: Inital Commit RAMPS FD v2.3. SPI Support for every Driver added.
Parts:
- C101: symbol CP1 -> RAMPS-FD-rescue:CP1
- C102, C207, C3, C4: symbol C -> RAMPS-FD-rescue:C
- D102: symbol DIODE_DUAL_ANODE -> RMC:DIODE_DUAL_ANODE
- D103: symbol D -> RAMPS-FD-rescue:D
- F101, F102, F103: symbol FUSE -> RAMPS-FD-rescue:FUSE
- J1: symbol NET-TIE -> RMC:NET-TIE
- JP1, JP201: symbol JUMP_MINI -> RMC:JUMP_MINI
- JP101, JP102: symbol JUMP_MINI_3 -> RMC:JUMP_MINI_3
- P101, P105: symbol CONN_2 -> RAMPS-FD-rescue:CONN_2
- P108: symbol CONN_4 -> RAMPS-FD-rescue:CONN_4
- P219: symbol CONN_3 -> RAMPS-FD-rescue:CONN_3
- U3: symbol LM7812 -> RAMPS-FD-rescue:LM7812
- U4: symbol LM7805 -> RAMPS-FD-rescue:LM7805
Connections:
- wire segments 81 -> 111

Commit message: Added UART for Communication with TMC2209 Drivers, improved inverse-polarity protection, added Driver Protection. Two Layer Design
Parts:
- removed C3, C4: 100n, Capacitors_SMD:C_0603, symbol RAMPS-FD-rescue:C
- removed D102: V10P10, rmc:TO277A_RMC, symbol RMC:DIODE_DUAL_ANODE
- removed P101: HB_IN, w_conn_screw:mstba_2,5%2f2-g-5,08, symbol RAMPS-FD-rescue:CONN_2
- removed P108: POWER_IN, w_conn_screw:mstba_2,5%2f4-g-5,08, symbol RAMPS-FD-rescue:CONN_4
- removed U4: L7805CV-DG, discret:LM78XXV, symbol RAMPS-FD-rescue:LM7805
- added D3, D4: KDZVTR11B, RAMPS-FD:D_SOD-123F, symbol RAMPS-FD:KDZVTR11B
- added F5, F6: FUSE_750mA_0603, RAMPS-FD:R_0603, symbol RAMPS-FD:FUSE_750mA_0603
- added J3: 6_PinScrewPlugableTerminal_P508, RAMPS-FD:6x1_P508_RA, symbol RAMPS-FD:6_PinScrewPlugableTerminal_P508
- added Q3, Q4: TDM3415, RAMPS-FD:SO-8_3.9x4.9mm_P1.27mm, symbol RAMPS-FD:TDM3415
- added R3, R4: 10k, RAMPS-FD:R_0603, symbol RAMPS-FD:10k
- C2: renamed from C101; value 100u 35V -> 100u_35V; footprint Capacitors_SMD:CP_Elec_6.3x7.7 -> RAMPS-FD:CP_Elec_6.3x7.7; symbol RAMPS-FD-rescue:CP1 -> RAMPS-FD:100u_35V; Fitted (none) -> yes; Ordering (none) -> LCSC: C88675; Price (USD) (none) -> 0,067122; Rating (none) -> #100uF #35V #20%
- C3: renamed from C102; value 100n 50V -> 100n; footprint Capacitors_SMD:C_0603 -> RAMPS-FD:C_0603; symbol RAMPS-FD-rescue:C -> RAMPS-FD:100n; Fitted (none) -> yes; Ordering (none) -> LCSC: C85999; Price (USD) (none) -> 0,016915; Rating (none) -> #100nF #50V #5%
- C4: renamed from C207; footprint Capacitors_SMD:C_0603 -> RAMPS-FD:C_0603; symbol RAMPS-FD-rescue:C -> RAMPS-FD:100n; Fitted (none) -> yes; Ordering (none) -> LCSC: C85999; Price (USD) (none) -> 0,016915; Rating (none) -> #100nF #50V #5%
- D5: renamed from D103; value ES1F -> MRA4003T3G; footprint rmc:DO-214AC -> RAMPS-FD:D_SMA; symbol RAMPS-FD-rescue:D -> RAMPS-FD:MRA4003T3G; Fitted (none) -> yes; Ordering (none) -> LCSC: C94410; Price (USD) (none) -> 0,049228; Rating (none) -> #300V #1A
- F2: renamed from F101; value FUSE 15A -> Keystone_3568; footprint rmc:Keystone_3568 -> RAMPS-FD:Fuseholder_Blade_Mini_Keystone_3568; symbol RAMPS-FD-rescue:FUSE -> RAMPS-FD:Keystone_3568; Fitted (none) -> yes; Ordering (none) -> Digikey: 36-3568-ND; Price (USD) (none) -> 1,03000; Rating (none) -> #500V #30A
- F3: renamed from F103; value FUSE 10A -> Keystone_3568; footprint rmc:Keystone_3568 -> RAMPS-FD:Fuseholder_Blade_Mini_Keystone_3568; symbol RAMPS-FD-rescue:FUSE -> RAMPS-FD:Keystone_3568; Fitted (none) -> yes; Ordering (none) -> Digikey: 36-3568-ND; Price (USD) (none) -> 1,03000; Rating (none) -> #500V #30A
- F4: renamed from F102; value FUSE 10A -> Keystone_3568; footprint rmc:Keystone_3568 -> RAMPS-FD:Fuseholder_Blade_Mini_Keystone_3568; symbol RAMPS-FD-rescue:FUSE -> RAMPS-FD:Keystone_3568; Fitted (none) -> yes; Ordering (none) -> Digikey: 36-3568-ND; Price (USD) (none) -> 1,03000; Rating (none) -> #500V #30A
- J4: renamed from J1; value NET-TIE -> NetTie_1mm; footprint rmc:TIE-1MM -> RAMPS-FD:TIE-1MM; symbol RMC:NET-TIE -> RAMPS-FD:NetTie_1mm
- J5: renamed from JP102; value VSEL -> 1x3JumperArray; footprint Pin_Headers:Pin_Header_Straight_1x03_Pitch2.54mm -> RAMPS-FD:PinHeader_1x03_P2.54mm_Vertical; symbol RMC:JUMP_MINI_3 -> RAMPS-FD:1x3JumperArray; Fitted (none) -> yes; Ordering (none) -> LCSC: C49257; Price (USD) (none) -> 0,010025
- J6: renamed from P105; value 12V-AUX -> 2x1PinHeader; footprint rmc:CONN_KK_2.54_2W -> RAMPS-FD:PinHeader_1x02_P2.54mm_Vertical; symbol RAMPS-FD-rescue:CONN_2 -> RAMPS-FD:2x1PinHeader; Fitted (none) -> yes; Ordering (none) -> LCSC: C124375; Price (USD) (none) -> 0,015147
- J7: renamed from JP101; value VLOG -> 1x3JumperArray; footprint Pin_Headers:Pin_Header_Straight_1x03_Pitch2.54mm -> RAMPS-FD:PinHeader_1x03_P2.54mm_Vertical; symbol RMC:JUMP_MINI_3 -> RAMPS-FD:1x3JumperArray; Fitted (none) -> yes; Ordering (none) -> LCSC: C49257; Price (USD) (none) -> 0,010025
- J8: renamed from P219; value EXT_5V -> 1x3PinHeader; footprint rmc:CONN_KK_2.54_3W -> RAMPS-FD:PinHeader_1x03_P2.54mm_Vertical; symbol RAMPS-FD-rescue:CONN_3 -> RAMPS-FD:1x3PinHeader; Fitted (none) -> yes; Ordering (none) -> LCSC: C49257; Price (USD) (none) -> 0,010025
- JP2: renamed from JP1; value VIN -> 1x2JumperArray; footprint Pin_Headers:Pin_Header_Straight_1x02_Pitch2.54mm -> RAMPS-FD:PinHeader_1x02_P2.54mm_Vertical; symbol RMC:JUMP_MINI -> RAMPS-FD:1x2JumperArray; Fitted (none) -> yes; Ordering (none) -> LCSC: C124375; Price (USD) (none) -> 0,015147
- JP3: renamed from JP201; value 5V_SEL -> 1x2JumperArray; footprint Pin_Headers:Pin_Header_Straight_1x02_Pitch2.54mm -> RAMPS-FD:PinHeader_1x02_P2.54mm_Vertical; symbol RMC:JUMP_MINI -> RAMPS-FD:1x2JumperArray; Fitted (none) -> yes; Ordering (none) -> LCSC: C124375; Price (USD) (none) -> 0,015147
- U2: renamed from U3; value R-78E12-0.5 -> AS7812ADTR; footprint discret:LM78XXV -> RAMPS-FD:TO-252-2; symbol RAMPS-FD-rescue:LM7812 -> RAMPS-FD:AS7812ADTR; Fitted (none) -> yes; Ordering (none) -> LCSC: C248312; Price (USD) (none) -> 0,203382; Rating (none) -> #12V #35V #1A
Connections:
- net labels removed: VCC
- wire segments 111 -> 122
Other:
- note removed: "or equivalent"
