File: RAMPS-FD/RAMPS-FD.sch (KiCad schematic (older format))
At the start: 11 parts, among them J2 CONN_02X06, M101 LOGO_OSHW, P102 RESET, Q101 DMN2075, SW101 RESET

Commit message: Inital Commit RAMPS FD v2.3. SPI Support for every Driver added.
Parts:
- removed J2: CONN_02X06, Pin_Headers:Pin_Header_Straight_2x06_Pitch2.54mm, symbol CONN_02X06
- D101: symbol LED-RESCUE-RAMPS-FD -> RAMPS-FD-rescue:LED-RESCUE-RAMPS-FD
- FID1, FID2, FID3: symbol Fiducial -> RMC:Fiducial
- M101: symbol LOGO_OSHW -> RMC:LOGO_OSHW
- P102: symbol CONN_2 -> RAMPS-FD-rescue:CONN_2
- Q101: symbol MOSFET_N -> RMC:MOSFET_N
- R101: symbol R -> RAMPS-FD-rescue:R
- SHIELD101: symbol ARDUINO_DUE_SHIELD -> RMC:ARDUINO_DUE_SHIELD
- SW101: symbol SW_PUSH -> RAMPS-FD-rescue:SW_PUSH
Connections:
- wire segments 96 -> 101
Changed lines of the file:
@@
-EESchema Schematic File Version 2
-LIBS:RAMPS-FD-rescue
-LIBS:power
-LIBS:device
-LIBS:transistors
-LIBS:conn
-LIBS:linear
-LIBS:regul
-LIBS:74xx
-LIBS:cmos4000
-LIBS:adc-dac
-LIBS:memory
-LIBS:xilinx
-LIBS:microcontrollers
-LIBS:dsp
-LIBS:microchip
-LIBS:analog_switches
-LIBS:motorola
-LIBS:texas
-LIBS:intel
-LIBS:audio
-LIBS:interface
-LIBS:digital-audio
-LIBS:philips
-LIBS:display
-LIBS:cypress
-LIBS:siliconi
-LIBS:opto
-LIBS:atmel
-LIBS:contrib
-LIBS:valves
-LIBS:RMC
-LIBS:RAMPS-FD-cache
-EELAYER 25 0
+EESchema Schematic File Version 4
+EELAYER 30 0
 EELAYER END
 $Descr A4 11693 8268
@@
 Sheet 1 10
 Title "RAMPS-FD (RAMPS for Arduino Due)"
-Date "2016-07-17"
-Rev "v2.2"
+Date "2019-04-13"
+Rev "v2.3"
 Comp ""
-Comment1 "Derived from RAMPS 1.4 reprap.org/wiki/RAMPS1.4"
+Comment1 "Derived from RAMPS FD 2.2 by Bob Cousins github.com/bobc/bobc_hardware/"
 Comment2 "GPL v3"
-Comment3 "Bob Cousins 2016"
+Comment3 "Marius Krause 2019"
 Comment4 ""
 $EndDescr
@@
 X/Y/Z pins are\non single port for both\nMega and Due
 $Comp
-L ARDUINO_DUE_SHIELD SHIELD101
+L RMC:ARDUINO_DUE_SHIELD SHIELD101
 U 1 1 50FC245D
 P 3200 3800
@@
 D11-FET4
 $Comp
-L LOGO_OSHW M101
+L RMC:LOGO_OSHW M101
 U 1 1 510E82F9
 P 6100 7200
@@
 	1    0    0    -1
 $EndComp
-Text GLabel 4350 4800 2    50   BiDi ~ 0
-D23
-Text GLabel 4350 5000 2    50   BiDi ~ 0
-D25
-Text GLabel 4350 5200 2    50   BiDi ~ 0
-D27
-Text GLabel 4350 5400 2    50   BiDi ~ 0
-D29
-Text GLabel 4350 5650 2    50   BiDi ~ 0
-D31
 Text GLabel 4350 5850 2    50   BiDi ~ 0
 D33
@@
 NoConn ~ 2200 6550
 $Comp
-L GND #PWR01
+L power:GND #PWR01
 U 1 1 51084806
 P 2200 6800
@@
 Z_DIR
 $Comp
-L PWR_FLAG #FLG02
+L power:PWR_FLAG #FLG02
 U 1 1 50FC2FBB
 P 1350 1950
@@
 Status LED
 $Comp
-L GND #PWR03
+L power:GND #PWR03
 U 1 1 50FC2571
 P 9500 5800
@@
 $EndComp
 $Comp
-L SW_PUSH SW101
+L RAMPS-FD-rescue:SW_PUSH SW101
 U 1 1 50FC254D
 P 9500 5100
@@
 RESET
 $Comp
-L GND #PWR04
+L power:GND #PWR04
 U 1 1 50FC24E2
 P 7950 5975
@@
 $EndComp
 $Comp
-L LED-RESCUE-RAMPS-FD D101
+L RAMPS-FD-rescue:LED-RESCUE-RAMPS-FD D101
 U 1 1 50FC24D8
 P 7950 4450
@@
 $EndComp
 $Comp
-L R R101
+L RAMPS-FD-rescue:R R101
 U 1 1 50FC24CE
 P 7950 5000
@@
 $EndComp
 $Comp
-L +3.3V #PWR05
+L power:+3.3V #PWR05
 U 1 1 50FC1A82
 P 1550 1700
@@
 $EndComp
 $Comp
-L GND #PWR06
+L power:GND #PWR06
 U 1 1 50FC1A69
 P 1400 2200
@@
 D13
 $Comp
-L CONN_2 P102
+L RAMPS-FD-rescue:CONN_2 P102
 U 1 1 52475D81
 P 10350 5100
@@
 NoConn ~ 4100 4500
 $Comp
-L GNDA #PWR07
+L power:GNDA #PWR07
 U 1 1 52CCBE6D
 P 1850 4550
@@
 $EndComp
 $Comp
-L PWR_FLAG #FLG08
+L power:PWR_FLAG #FLG08
 U 1 1 52CCBF6C
 P 1650 4400
@@
 $EndComp
 $Comp
-L +5V #PWR09
+L power:+5V #PWR09
 U 1 1 52D057D7
 P 7950 4050
@@
 $EndComp
 $Comp
-L MOSFET_N Q101
+L RMC:MOSFET_N Q101
 U 1 1 52D0586E
 P 7875 5550
@@
 	4100 6250 4350 6250
 Wire Wire Line
-	4100 5850 4350 5850
-Wire Wire Line
-	4100 5650 4350 5650
-Wire Wire Line
-	4100 5200 4350 5200
-Wire Wire Line
-	4100 4800 4350 4800
-Wire Wire Line
 	1000 5950 2200 5950
 Wire Wire Line
@@
 	1000 5400 2200 5400
 Wire Wire Line
-	1350 1950 2200 1950
+	1350 1950 1550 1950
 Wire Wire Line
 	4100 6150 5200 6150
@@
 	2200 2550 1450 2550
 Wire Wire Line
-	9500 5400 9500 5800
+	9500 5400 9500 5700
 Wire Wire Line
 	7100 5625 7575 5625
@@
 	1000 6150 2200 6150
 Wire Wire Line
-	4100 5000 4350 5000
-Wire Wire Line
-	4100 5400 4350 5400
-Wire Wire Line
 	4100 5750 5200 5750
 Wire Wire Line
@@
 	1450 6050 2200 6050
 Wire Wire Line
-	9150 4600 9950 4600
+	9150 4600 9500 4600
 Wire Wire Line
 	9500 4600 9500 4800
@@
 	2200 4500 1850 4500
 Wire Wire Line
-	1850 4400 1850 4550
-Wire Wire Line
-	1650 4400 2200 4400
+	1850 4400 1850 4500
+Wire Wire Line
+	1650 4400 1850 4400
 Connection ~ 1850 4500
 Connection ~ 1850 4400
@@
 LED
 $Comp
-L Fiducial FID2
+L RMC:Fiducial FID2
 U 1 1 5725214B
 P 10375 3975
@@
 $EndComp
 $Comp
-L Fiducial FID3
+L RMC:Fiducial FID3
 U 1 1 572521B8
 P 10775 3975
@@
 $EndComp
 $Comp
-L Fiducial FID1
+L RMC:Fiducial FID1
 U 1 1 57252215
 P 10000 3975
@@
 	1    0    0    -1
 $EndComp
-Text GLabel 4800 7200 2    50   Output ~ 0
+Text GLabel 1850 3250 2    50   Output ~ 0
 STEP_Y_CS
-$Comp
-L CONN_02X06 J2
-U 1 1 5B124015
-P 4550 7350
-F 0 "J2" H 4550 7700 50  0000 C CNN
-F 1 "CONN_02X06" H 4550 7000 50  0000 C CNN
-F 2 "Pin_Headers:Pin_Header_Straight_2x06_Pitch2.54mm" H 4550 6150 50  0001 C CNN
-F 3 "" H 4550 6150 50  0001 C CNN
-	1    4550 7350
-	1    0    0    -1
-$EndComp
-Text GLabel 4800 7100 2    50   Output ~ 0
+Text GLabel 1000 4150 2    50   Output ~ 0
 STEP_X_CS
-Text GLabel 4800 7300 2    50   Output ~ 0
+Text GLabel 1850 3150 2    50   Output ~ 0
 STEP_Z_CS
-Text GLabel 4800 7400 2    50   Output ~ 0
+Text GLabel 1850 2950 2    50   Output ~ 0
 STEP_E0_CS
-Text GLabel 4800 7500 2    50   Output ~ 0
+Text GLabel 1850 3050 2    50   Output ~ 0
 STEP_E1_CS
-Text GLabel 4800 7600 2    50   Output ~ 0
+Text GLabel 1000 4050 2    50   Output ~ 0
 STEP_E2_CS
-Text GLabel 4300 7600 0    50   BiDi ~ 0
-D33
-Text GLabel 4300 7500 0    50   BiDi ~ 0
+Wire Wire Line
+	1550 1950 2200 1950
+Wire Wire Line
+	9500 4600 9950 4600
+Wire Wire Line
+	9500 5700 9500 5800
+Wire Wire Line
+	1850 4500 1850 4550
+Wire Wire Line
+	1850 4400 2200 4400
+Text GLabel 4350 5650 2    50   BiDi ~ 0
 D31
-Text GLabel 4300 7400 0    50   BiDi ~ 0
+Text GLabel 4350 5400 2    50   BiDi ~ 0
 D29
-Text GLabel 4300 7300 0    50   BiDi ~ 0
+Text GLabel 4350 5200 2    50   BiDi ~ 0
 D27
-Text GLabel 4300 7200 0    50   BiDi ~ 0
+Text GLabel 4350 5000 2    50   BiDi ~ 0
 D25
-Text GLabel 4300 7100 0    50   BiDi ~ 0
+Text GLabel 4350 4800 2    50   BiDi ~ 0
 D23
+Wire Wire Line
+	4100 4800 4750 4800
+Wire Wire Line
+	4100 5000 4750 5000
+Wire Wire Line
+	4100 5200 4750 5200
+Wire Wire Line
+	4100 5400 4750 5400
+Wire Wire Line
+	4100 5650 4750 5650
+Wire Wire Line
+	4100 5850 4750 5850
 $EndSCHEMATC

Commit message: Added UART for Communication with TMC2209 Drivers, improved inverse-polarity protection, added Driver Protection. Two Layer Design
Parts:
- removed R101: 330R, Resistors_SMD:R_0603, symbol RAMPS-FD-rescue:R
- added R2: 330R, RAMPS-FD:R_0603, symbol RAMPS-FD:330R
- D2: renamed from D101; value STATUS -> LED_0603_GREEN; footprint rmc:LED-0805_GREEN -> RAMPS-FD:LED_0603; symbol RAMPS-FD-rescue:LED-RESCUE-RAMPS-FD -> RAMPS-FD:LED_0603_GREEN; Fitted (none) -> yes; Ordering (none) -> LCSC: C192316; Price (USD) (none) -> 0,021656
- FID2: renamed from FID1; footprint Fiducials:Fiducial_1mm_Dia_2.54mm_Outer_CopperTop -> RAMPS-FD:Fiducial_1mm_Mask2mm; symbol RMC:Fiducial -> RAMPS-FD:Fiducial
- FID3: renamed from FID2; footprint Fiducials:Fiducial_1mm_Dia_2.54mm_Outer_CopperTop -> RAMPS-FD:Fiducial_1mm_Mask2mm; symbol RMC:Fiducial -> RAMPS-FD:Fiducial
- FID4: renamed from FID3; footprint Fiducials:Fiducial_1mm_Dia_2.54mm_Outer_CopperTop -> RAMPS-FD:Fiducial_1mm_Mask2mm; symbol RMC:Fiducial -> RAMPS-FD:Fiducial
- J2: renamed from P102; value RESET -> 2x1PinHeader; footprint Pin_Headers:Pin_Header_Straight_1x02_Pitch2.54mm -> RAMPS-FD:PinHeader_1x02_P2.54mm_Vertical; symbol RAMPS-FD-rescue:CONN_2 -> RAMPS-FD:2x1PinHeader; Fitted (none) -> yes; Ordering (none) -> LCSC: C124375; Price (USD) (none) -> 0,015147
- M2: renamed from M101; footprint rmc:OSHW_logo_2 -> RAMPS-FD:OSHW_logo_2; symbol RMC:LOGO_OSHW -> RAMPS-FD:LOGO_OSHW
- Q2: renamed from Q101; value DMN2075 -> NCE3416; footprint libcms:SOT23GDS -> RAMPS-FD:SOT-23; symbol RMC:MOSFET_N -> RAMPS-FD:NCE3416; Fitted (none) -> yes; Ordering (none) -> LCSC: C113491; Price (USD) (none) -> 0,033091; Rating (none) -> #20V #6.5A
- SHIELD2: renamed from SHIELD101; footprint rmc:ARDUINO_MEGA_DUE_SHIELD_FOOTPRINT_RMC -> RAMPS-FD:ARDUINO_MEGA_DUE_SHIELD_FOOTPRINT_RMC; symbol RMC:ARDUINO_DUE_SHIELD -> RAMPS-FD:ARDUINO_DUE_SHIELD; Fitted (none) -> yes; Ordering (none) -> LCSC: 1xC124372 5xC124381 1xC168945
- SW2: renamed from SW101; value RESET -> PushButton; footprint rmc:SW_6x6_SMD -> RAMPS-FD:SW_6x6_SMD; symbol RAMPS-FD-rescue:SW_PUSH -> RAMPS-FD:PushButton; Fitted (none) -> yes; Ordering (none) -> LCSC: C273496; Price (USD) (none) -> 0,497955
Connections:
- wire segments 101 -> 102
Changed lines of the file:
@@
 X/Y/Z pins are\non single port for both\nMega and Due
 $Comp
-L RMC:ARDUINO_DUE_SHIELD SHIELD101
+L RAMPS-FD:ARDUINO_DUE_SHIELD SHIELD2
 U 1 1 50FC245D
 P 3200 3800
-F 0 "SHIELD101" H 2800 6650 60  0000 C CNN
+F 0 "SHIELD2" H 2800 6650 60  0000 C CNN
 F 1 "ARDUINO_DUE_SHIELD" H 3150 750 60  0000 C CNN
-F 2 "rmc:ARDUINO_MEGA_DUE_SHIELD_FOOTPRINT_RMC" H 3200 3800 60  0001 C CNN
+F 2 "RAMPS-FD:ARDUINO_MEGA_DUE_SHIELD_FOOTPRINT_RMC" H 3200 3800 60  0001 C CNN
 F 3 "" H 3200 3800 60  0001 C CNN
+F 4 "yes" H 0   0   50  0001 C CNN "Fitted"
+F 5 "LCSC: 1xC124372 5xC124381 1xC168945" H 0   0   50  0001 C CNN "Ordering"
 	1    3200 3800
 	1    0    0    -1
@@
 D11-FET4
 $Comp
-L RMC:LOGO_OSHW M101
+L RAMPS-FD:LOGO_OSHW M2
 U 1 1 510E82F9
 P 6100 7200
-F 0 "M101" H 6100 7350 60  0000 C CNN
+F 0 "M2" H 6100 7350 60  0000 C CNN
 F 1 "LOGO_OSHW" H 6100 7100 60  0000 C CNN
-F 2 "rmc:OSHW_logo_2" H 6000 7250 60  0001 C CNN
+F 2 "RAMPS-FD:OSHW_logo_2" H 6000 7250 60  0001 C CNN
 F 3 "" H 6100 7200 60  0001 C CNN
 F 4 "No" H 6100 7200 60  0001 C CNN "Populate"
@@
 NoConn ~ 2200 6550
 $Comp
-L power:GND #PWR01
+L power:GND #PWR08
 U 1 1 51084806
 P 2200 6800
-F 0 "#PWR01" H 2200 6800 30  0001 C CNN
+F 0 "#PWR08" H 2200 6800 30  0001 C CNN
 F 1 "GND" H 2200 6730 30  0001 C CNN
 F 2 "" H 2200 6800 60  0001 C CNN
@@
 F 1 "PWR_FLAG" H 1350 2130 30  0000 C CNN
 F 2 "" H 1350 1950 60  0001 C CNN
-F 3 "" H 1350 1950 60  0001 C CNN
+F 3 "~" H 1350 1950 60  0001 C CNN
 	1    1350 1950
 	1    0    0    -1
@@
 Status LED
 $Comp
-L power:GND #PWR03
+L power:GND #PWR06
 U 1 1 50FC2571
 P 9500 5800
-F 0 "#PWR03" H 9500 5800 30  0001 C CNN
+F 0 "#PWR06" H 9500 5800 30  0001 C CNN
 F 1 "GND" H 9500 5730 30  0001 C CNN
 F 2 "" H 9500 5800 60  0001 C CNN
@@
 $EndComp
 $Comp
-L RAMPS-FD-rescue:SW_PUSH SW101
+L RAMPS-FD:PushButton SW2
 U 1 1 50FC254D
 P 9500 5100
-F 0 "SW101" H 9500 5250 50  0000 C CNN
-F 1 "RESET" H 9500 5020 50  0000 C CNN
-F 2 "rmc:SW_6x6_SMD" H 9500 5100 60  0001 C CNN
+F 0 "SW2" H 9500 5250 50  0000 C CNN
+F 1 "PushButton" H 9500 5020 50  0000 C CNN
+F 2 "RAMPS-FD:SW_6x6_SMD" H 9500 5100 60  0001 C CNN
 F 3 "" H 9500 5100 60  0001 C CNN
+F 4 "yes" H 0   0   50  0001 C CNN "Fitted"
+F 5 "LCSC: C273496" H 0   0   50  0001 C CNN "Ordering"
+F 6 "0,497955" H 0   0   50  0001 C CNN "Price (USD)"
 	1    9500 5100
 	0    -1   1    0
@@
 RESET
 $Comp
-L power:GND #PWR04
+L power:GND #PWR07
 U 1 1 50FC24E2
-P 7950 5975
-F 0 "#PWR04" H 7950 5975 30  0001 C CNN
-F 1 "GND" H 7950 5905 30  0001 C CNN
-F 2 "" H 7950 5975 60  0001 C CNN
-F 3 "" H 7950 5975 60  0001 C CNN
-	1    7950 5975
-	1    0    0    -1
-$EndComp
-$Comp
-L RAMPS-FD-rescue:LED-RESCUE-RAMPS-FD D101
+P 7950 6000
+F 0 "#PWR07" H 7950 6000 30  0001 C CNN
+F 1 "GND" H 7950 5930 30  0001 C CNN
+F 2 "" H 7950 6000 60  0001 C CNN
+F 3 "" H 7950 6000 60  0001 C CNN
+	1    7950 6000
+	1    0    0    -1
+$EndComp
+$Comp
+L RAMPS-FD:LED_0603_GREEN D2
 U 1 1 50FC24D8
 P 7950 4450
-F 0 "D101" H 7950 4550 50  0000 C CNN
-F 1 "STATUS" H 7950 4300 50  0000 C CNN
-F 2 "rmc:LED-0805_GREEN" H 7950 4450 60  0001 C CNN
-F 3 "" H 7950 4450 60  0001 C CNN
+F 0 "D2" H 7950 4550 50  0000 C CNN
+F 1 "LED_0603_GREEN" H 7950 4300 50  0000 C CNN
+F 2 "RAMPS-FD:LED_0603" H 7950 4450 60  0001 C CNN
+F 3 "https://datasheet.lcsc.com/szlcsc/1811141223_TOGIALED-TJ-S1608SW6TGLC2G-A5_C192316.pdf" H 7950 4450 60  0001 C CNN
+F 4 "yes" H 0   0   50  0001 C CNN "Fitted"
+F 5 "LCSC: C192316" H 0   0   50  0001 C CNN "Ordering"
+F 6 "0,021656" H 0   0   50  0001 C CNN "Price (USD)"
 	1    7950 4450
 	0    -1   -1   0
 $EndComp
 $Comp
-L RAMPS-FD-rescue:R R101
-U 1 1 50FC24CE
-P 7950 5000
-F 0 "R101" V 8050 5000 50  0000 C CNN
-F 1 "330R" V 7950 5000 50  0000 C CNN
-F 2 "Resistors_SMD:R_0603" H 7950 5000 60  0001 C CNN
-F 3 "" H 7950 5000 60  0001 C CNN
-	1    7950 5000
-	1    0    0    -1
-$EndComp
-$Comp
-L power:+3.3V #PWR05
+L power:+3.3V #PWR02
 U 1 1 50FC1A82
 P 1550 1700
-F 0 "#PWR05" H 1550 1660 30  0001 C CNN
+F 0 "#PWR02" H 1550 1660 30  0001 C CNN
 F 1 "+3.3V" H 1550 1810 30  0000 C CNN
 F 2 "" H 1550 1700 60  0001 C CNN
@@
 $EndComp
 $Comp
-L power:GND #PWR06
+L power:GND #PWR03
 U 1 1 50FC1A69
 P 1400 2200
-F 0 "#PWR06" H 1400 2200 30  0001 C CNN
+F 0 "#PWR03" H 1400 2200 30  0001 C CNN
 F 1 "GND" H 1400 2130 30  0001 C CNN
 F 2 "" H 1400 2200 60  0001 C CNN
@@
 D13
 $Comp
-L RAMPS-FD-rescue:CONN_2 P102
+L RAMPS-FD:2x1PinHeader J2
 U 1 1 52475D81
-P 10350 5100
-F 0 "P102" V 10300 5100 40  0000 C CNN
-F 1 "RESET" V 10400 5100 40  0000 C CNN
-F 2 "Pin_Headers:Pin_Header_Straight_1x02_Pitch2.54mm" H 10350 5100 60  0001 C CNN
-F 3 "" H 10350 5100 60  0000 C CNN
-	1    10350 5100
+P 10250 5050
+F 0 "J2" H 10250 5150 40  0000 C CNN
+F 1 "2x1PinHeader" H 10250 4850 40  0000 C CNN
+F 2 "RAMPS-FD:PinHeader_1x02_P2.54mm_Vertical" H 10250 5050 60  0001 C CNN
+F 3 "" H 10250 5050 60  0000 C CNN
+F 4 "yes" H 0   0   50  0001 C CNN "Fitted"
+F 5 "LCSC: C124375" H 0   0   50  0001 C CNN "Ordering"
+F 6 "0,015147" H 0   0   50  0001 C CNN "Price (USD)"
+	1    10250 5050
 	1    0    0    -1
 $EndComp
@@
 NoConn ~ 4100 4500
 $Comp
-L power:GNDA #PWR07
+L power:GNDA #PWR05
 U 1 1 52CCBE6D
 P 1850 4550
-F 0 "#PWR07" H 1850 4300 50  0001 C CNN
+F 0 "#PWR05" H 1850 4300 50  0001 C CNN
 F 1 "GNDA" H 1850 4400 50  0000 C CNN
 F 2 "" H 1850 4550 50  0000 C CNN
@@
 $EndComp
 $Comp
-L power:PWR_FLAG #FLG08
+L power:PWR_FLAG #FLG03
 U 1 1 52CCBF6C
 P 1650 4400
-F 0 "#FLG08" H 1650 4495 30  0001 C CNN
+F 0 "#FLG03" H 1650 4495 30  0001 C CNN
 F 1 "PWR_FLAG" H 1650 4580 30  0000 C CNN
 F 2 "" H 1650 4400 60  0001 C CNN
-F 3 "" H 1650 4400 60  0001 C CNN
+F 3 "~" H 1650 4400 60  0001 C CNN
 	1    1650 4400
 	1    0    0    -1
 $EndComp
 $Comp
-L power:+5V #PWR09
+L power:+5V #PWR04
 U 1 1 52D057D7
 P 7950 4050
-F 0 "#PWR09" H 7950 3900 50  0001 C CNN
+F 0 "#PWR04" H 7950 3900 50  0001 C CNN
 F 1 "+5V" H 7950 4190 50  0000 C CNN
 F 2 "" H 7950 4050 50  0000 C CNN
@@
 	1    0    0    -1
 $EndComp
-$Comp
-L RMC:MOSFET_N Q101
-U 1 1 52D0586E
-P 7875 5550
-F 0 "Q101" H 7875 5750 60  0000 R CNN
-F 1 "DMN2075" H 7875 5300 60  0000 R CNN
-F 2 "libcms:SOT23GDS" H 7875 5550 60  0001 C CNN
-F 3 "~" H 7875 5550 60  0000 C CNN
-	1    7875 5550
-	1    0    0    -1
-$EndComp
 NoConn ~ 4100 1450
 Wire Wire Line
@@
 Wire Wire Line
 	9500 5400 9500 5700
-Wire Wire Line
-	7100 5625 7575 5625
-Wire Wire Line
-	7950 5825 7950 5975
 Wire Wire Line
 	1550 1950 1550 1700
@@
 Wire Notes Line
 	5650 2650 5900 2650
-Wire Wire Line
-	9950 4600 9950 5000
-Wire Wire Line
-	9950 5000 10000 5000
 Connection ~ 9500 4600
-Wire Wire Line
-	10000 5200 10000 5700
 Wire Wire Line
 	10000 5700 9500 5700
@@
 Connection ~ 1850 4500
 Connection ~ 1850 4400
-Wire Wire Line
-	7950 4050 7950 4250
-Wire Wire Line
-	7950 5275 7950 5150
-Text GLabel 7100 5625 0    50   Input ~ 0
+Text GLabel 7200 5600 0    50   Input ~ 0
 D13
 Text Notes 5250 1650 0    60   ~ 0
 LED
 $Comp
-L RMC:Fiducial FID2
+L RAMPS-FD:Fiducial FID3
 U 1 1 5725214B
 P 10375 3975
-F 0 "FID2" H 10375 3775 60  0000 C CNN
+F 0 "FID3" H 10375 3775 60  0000 C CNN
 F 1 "Fiducial" H 10375 4125 60  0000 C CNN
-F 2 "Fiducials:Fiducial_1mm_Dia_2.54mm_Outer_CopperTop" H 10275 3675 60  0001 C CNN
+F 2 "RAMPS-FD:Fiducial_1mm_Mask2mm" H 10275 3675 60  0001 C CNN
 F 3 "" H 10375 3975 60  0000 C CNN
 F 4 "No" H 10375 3975 60  0001 C CNN "Populate"
@@
 $EndComp
 $Comp
-L RMC:Fiducial FID3
+L RAMPS-FD:Fiducial FID4
 U 1 1 572521B8
 P 10775 3975
-F 0 "FID3" H 10775 3775 60  0000 C CNN
+F 0 "FID4" H 10775 3775 60  0000 C CNN
 F 1 "Fiducial" H 10775 4125 60  0000 C CNN
-F 2 "Fiducials:Fiducial_1mm_Dia_2.54mm_Outer_CopperTop" H 10675 3675 60  0001 C CNN
+F 2 "RAMPS-FD:Fiducial_1mm_Mask2mm" H 10675 3675 60  0001 C CNN
 F 3 "" H 10775 3975 60  0000 C CNN
 F 4 "No" H 10775 3975 60  0001 C CNN "Populate"
@@
 $EndComp
 $Comp
-L RMC:Fiducial FID1
+L RAMPS-FD:Fiducial FID2
 U 1 1 57252215
 P 10000 3975
-F 0 "FID1" H 10000 3775 60  0000 C CNN
+F 0 "FID2" H 10000 3775 60  0000 C CNN
 F 1 "Fiducial" H 10000 4125 60  0000 C CNN
-F 2 "Fiducials:Fiducial_1mm_Dia_2.54mm_Outer_CopperTop" H 9900 3675 60  0001 C CNN
+F 2 "RAMPS-FD:Fiducial_1mm_Mask2mm" H 9900 3675 60  0001 C CNN
 F 3 "" H 10000 3975 60  0000 C CNN
 F 4 "No" H 10000 3975 60  0001 C CNN "Populate"
@@
 Wire Wire Line
 	4100 5850 4750 5850
+$Comp
+L RAMPS-FD:330R R2
+U 1 1 5EFEC45D
+P 7950 5000
+F 0 "R2" V 8025 4950 50  0000 L CNN
+F 1 "330R" V 7950 4900 50  0000 L CNN
+F 2 "RAMPS-FD:R_0603" V 7880 5000 50  0001 C CNN
+F 3 "" H 7950 5000 50  0001 C CNN
+F 4 "yes" H 0   0   50  0001 C CNN "Fitted"
+F 5 "LCSC: C144606" H 0   0   50  0001 C CNN "Ordering"
+F 6 "0,002275" H 0   0   50  0001 C CNN "Price (USD)"
+	1    7950 5000
+	1    0    0    -1
+$EndComp
+Wire Wire Line
+	7950 4050 7950 4350
+$Comp
+L RAMPS-FD:NCE3416 Q2
+U 1 1 52D0586E
+P 7550 5600
+F 0 "Q2" H 7700 5850 60  0000 R CNN
+F 1 "NCE3416" H 7900 5400 60  0000 R CNN
+F 2 "RAMPS-FD:SOT-23" H 7550 5600 60  0001 C CNN
+F 3 "https://datasheet.lcsc.com/szlcsc/1811071721_Wuxi-NCE-Power-Semiconductor-NCE3416_C113491.pdf" H 7550 5600 60  0001 C CNN
+F 4 "#20V #6.5A" H 7550 5600 50  0001 C CNN "Rating"
+F 5 "yes" H 0   0   50  0001 C CNN "Fitted"
+F 6 "LCSC: C113491 " H 0   0   50  0001 C CNN "Ordering"
+F 7 "0,033091" H 0   0   50  0001 C CNN "Price (USD)"
+	1    7550 5600
+	1    0    0    -1
+$EndComp
+Wire Wire Line
+	7550 5600 7200 5600
+Wire Wire Line
+	7950 5250 7950 5150
+Wire Wire Line
+	7950 5800 7950 6000
+Wire Wire Line
+	10200 5050 9950 5050
+Wire Wire Line
+	10000 5150 10200 5150
+Wire Wire Line
+	10000 5150 10000 5700
+Wire Wire Line
+	9950 4600 9950 5050
 $EndSCHEMATC
