File: RAMPS-FD/con_misc.sch (KiCad schematic (older format))
At the start: 17 parts, among them K201 S1, K202 S2, K203 S3, K204 S4, P1 SERIAL1, P2 I2C-1, P211 I2C-0, P213 AUX-4, P214 AUX-2, P215 AUX-3, P216 SERIAL0, U601 24C512

Commit message: Inital Commit RAMPS FD v2.3. SPI Support for every Driver added.
Parts:
- C601: symbol C -> RAMPS-FD-rescue:C
- K201, K202, K203, K204: symbol CONN_3 -> RAMPS-FD-rescue:CONN_3
- P1, P216: symbol CONN_6 -> RAMPS-FD-rescue:CONN_6
- P2, P211: symbol CONN_4 -> RAMPS-FD-rescue:CONN_4
- P213: symbol CONN_18 -> RMC:CONN_18
- P214: symbol CONN_5X2 -> RAMPS-FD-rescue:CONN_5X2
- P215: symbol CONN_6X2 -> RAMPS-FD-rescue:CONN_6X2
- R1, R2, R211, R212: symbol R -> RAMPS-FD-rescue:R
- U601: symbol 24C512 -> RAMPS-FD-rescue:24C512
Connections:
- wire segments 108 -> 120
Changed lines of the file:
@@
-EESchema Schematic File Version 2
-LIBS:RAMPS-FD-rescue
-LIBS:power
-LIBS:device
-LIBS:transistors
-LIBS:conn
-LIBS:linear
-LIBS:regul
-LIBS:74xx
-LIBS:cmos4000
-LIBS:adc-dac
-LIBS:memory
-LIBS:xilinx
-LIBS:microcontrollers
-LIBS:dsp
-LIBS:microchip
-LIBS:analog_switches
-LIBS:motorola
-LIBS:texas
-LIBS:intel
-LIBS:audio
-LIBS:interface
-LIBS:digital-audio
-LIBS:philips
-LIBS:display
-LIBS:cypress
-LIBS:siliconi
-LIBS:opto
-LIBS:atmel
-LIBS:contrib
-LIBS:valves
-LIBS:RMC
-LIBS:RAMPS-FD-cache
-EELAYER 25 0
+EESchema Schematic File Version 4
+EELAYER 30 0
 EELAYER END
 $Descr A4 11693 8268
@@
 Sheet 6 10
 Title "RAMPS-FD (RAMPS for Arduino Due)"
-Date "2016-07-17"
-Rev "v2.2"
+Date "2019-04-13"
+Rev "v2.3"
 Comp ""
-Comment1 "Derived from RAMPS 1.4 reprap.org/wiki/RAMPS1.4"
+Comment1 "Derived from RAMPS FD 2.2 by Bob Cousins github.com/bobc/bobc_hardware/"
 Comment2 "GPL v3"
-Comment3 "Bob Cousins 2016"
+Comment3 "Marius Krause 2019"
 Comment4 ""
 $EndDescr
@@
 	4450 2150 4450 2500
 Wire Wire Line
-	4250 2400 5450 2400
+	4250 2400 4800 2400
 Connection ~ 4800 1650
 Wire Wire Line
 	4800 1850 4800 1650
 Wire Wire Line
-	4450 1650 5250 1650
+	4450 1650 4800 1650
 Wire Wire Line
 	5250 1650 5250 2200
@@
 	5250 2200 5450 2200
 Wire Wire Line
-	4450 1600 4450 1850
+	4450 1600 4450 1650
 Connection ~ 4450 1650
 Wire Wire Line
@@
 	5250 2300 5250 2600
 Wire Wire Line
-	4250 2500 5450 2500
+	4250 2500 4450 2500
 Wire Wire Line
 	1350 4400 1700 4400
@@
 	1950 2800 1950 3600
 Wire Wire Line
-	4250 4700 5450 4700
+	4250 4700 4450 4700
 Wire Wire Line
 	5250 4800 5250 4500
@@
 Connection ~ 4450 3850
 Wire Wire Line
-	4450 3800 4450 4050
+	4450 3800 4450 3850
 Wire Wire Line
 	5450 4400 5250 4400
@@
 	5250 4400 5250 3850
 Wire Wire Line
-	5250 3850 4450 3850
+	5250 3850 4800 3850
 Wire Wire Line
 	4800 4050 4800 3850
 Connection ~ 4800 3850
 Wire Wire Line
-	4250 4600 5450 4600
+	4250 4600 4800 4600
 Wire Wire Line
 	4450 4350 4450 4700
@@
 D52-SCK
 $Comp
-L CONN_4 P2
+L RAMPS-FD-rescue:CONN_4 P2
 U 1 1 523B6020
 P 5800 4550
@@
 $EndComp
 $Comp
-L R R2
+L RAMPS-FD-rescue:R R2
 U 1 1 523B601F
 P 4800 4200
@@
 $EndComp
 $Comp
-L R R1
+L RAMPS-FD-rescue:R R1
 U 1 1 523B601E
 P 4450 4200
@@
 $EndComp
 $Comp
-L GND #PWR071
+L power:GND #PWR071
 U 1 1 523B601D
 P 5250 4800
@@
 SCL1
 $Comp
-L +V_LOGIC #PWR071
+L RMC:+V_LOGIC #PWR071
 U 1 1 523B601C
 P 4450 3800
@@
 UART1_TX_LV
 $Comp
-L GND #PWR073
+L power:GND #PWR073
 U 1 1 523B5AB9
 P 1950 3600
@@
 $EndComp
 $Comp
-L CONN_6 P1
+L RAMPS-FD-rescue:CONN_6 P1
 U 1 1 523B5AB8
 P 2800 3050
@@
 NoConn ~ 2450 1650
 $Comp
-L CONN_6 P216
+L RAMPS-FD-rescue:CONN_6 P216
 U 1 1 51F17B03
 P 2800 1800
@@
 D51-MOSI
 $Comp
-L +V_LOGIC #PWR073
+L RMC:+V_LOGIC #PWR073
 U 1 1 517867DD
 P 7950 1750
@@
 $EndComp
 $Comp
-L +V_LOGIC #PWR074
+L RMC:+V_LOGIC #PWR074
 U 1 1 517867D0
 P 8250 6475
@@
 $EndComp
 $Comp
-L +V_LOGIC #PWR075
+L RMC:+V_LOGIC #PWR075
 U 1 1 517867C6
 P 4450 1600
@@
 $EndComp
 $Comp
-L GND #PWR077
+L power:GND #PWR077
 U 1 1 51084B2C
 P 9100 6425
@@
 D23
 $Comp
-L CONN_18 P213
+L RMC:CONN_18 P213
 U 1 1 51084A74
 P 9700 5575
@@
 Must not have external pullups to 5V if IOREF = 3.3V
 $Comp
-L GND #PWR078
+L power:GND #PWR078
 U 1 1 5104884C
 P 7550 3600
@@
 $EndComp
 $Comp
-L GND #PWR079
+L power:GND #PWR079
 U 1 1 51048839
 P 10000 1900
@@
 $EndComp
 $Comp
-L GND #PWR080
+L power:GND #PWR080
 U 1 1 5104861F
 P 1950 2350
@@
 Servos
 $Comp
-L CONN_5X2 P214
+L RAMPS-FD-rescue:CONN_5X2 P214
 U 1 1 510481EC
 P 8850 2050
@@
 $EndComp
 $Comp
-L CONN_3 K204
+L RAMPS-FD-rescue:CONN_3 K204
 U 1 1 51047C7F
 P 2050 6650
@@
 $EndComp
 $Comp
-L GND #PWR081
+L power:GND #PWR081
 U 1 1 51047C7E
 P 1550 6850
@@
 $EndComp
 $Comp
-L +5V #PWR081
+L power:+5V #PWR081
 U 1 1 51047C7D
 P 1550 6450
@@
 SERVO3
 $Comp
-L +5V #PWR082
+L power:+5V #PWR082
 U 1 1 51047C7B
 P 1550 5700
@@
 $EndComp
 $Comp
-L GND #PWR084
+L power:GND #PWR084
 U 1 1 51047C7A
 P 1550 6100
@@
 $EndComp
 $Comp
-L CONN_3 K203
+L RAMPS-FD-rescue:CONN_3 K203
 U 1 1 51047C79
 P 2050 5900
@@
 $EndComp
 $Comp
-L CONN_3 K202
+L RAMPS-FD-rescue:CONN_3 K202
 U 1 1 51047C78
 P 2050 5250
@@
 $EndComp
 $Comp
-L GND #PWR085
+L power:GND #PWR085
 U 1 1 51047C77
 P 1550 5450
@@
 $EndComp
 $Comp
-L +5V #PWR085
+L power:+5V #PWR085
 U 1 1 51047C76
 P 1550 5050
@@
 SERVO1
 $Comp
-L +5V #PWR086
+L power:+5V #PWR086
 U 1 1 51047C09
 P 1550 4300
@@
 $EndComp
 $Comp
-L GND #PWR088
+L power:GND #PWR088
 U 1 1 51047C01
 P 1550 4700
@@
 $EndComp
 $Comp
-L CONN_3 K201
+L RAMPS-FD-rescue:CONN_3 K201
 U 1 1 51047BDF
 P 2050 4500
@@
 SDA
 $Comp
-L GND #PWR089
+L power:GND #PWR089
 U 1 1 51047413
 P 5250 2600
@@
 $EndComp
 $Comp
-L R R211
+L RAMPS-FD-rescue:R R211
 U 1 1 510473D0
 P 4450 2000
@@
 $EndComp
 $Comp
-L R R212
+L RAMPS-FD-rescue:R R212
 U 1 1 510473CD
 P 4800 2000
@@
 $EndComp
 $Comp
-L CONN_4 P211
+L RAMPS-FD-rescue:CONN_4 P211
 U 1 1 51047175
 P 5800 2350
@@
 	9400 5725 8050 5725
 $Comp
-L +5V #PWR089
+L power:+5V #PWR089
 U 1 1 52421C84
 P 7950 3100
@@
 NoConn ~ 9250 3500
 $Comp
-L CONN_6X2 P215
+L RAMPS-FD-rescue:CONN_6X2 P215
 U 1 1 52475600
 P 8850 3450
@@
 $EndComp
 $Comp
-L +V_LOGIC #PWR090
+L RMC:+V_LOGIC #PWR090
 U 1 1 52475621
 P 10250 3650
@@
 Note: Some addon boards \nconnect this pin to GND.
 $Comp
-L 24C512 U601
+L RAMPS-FD-rescue:24C512 U601
 U 1 1 52B23647
 P 4400 6250
+AR Path="/52B23647" Ref="U601"  Part="1"
+AR Path="/5176EFAC/52B23647" Ref="U601"  Part="1"
 F 0 "U601" H 4550 6600 60  0000 C CNN
 F 1 "24C512" H 4600 5900 60  0000 C CNN
@@
 $EndComp
 $Comp
-L GND #PWR092
+L power:GND #PWR092
 U 1 1 52B23654
 P 4400 6900
@@
 $EndComp
 Wire Wire Line
-	4400 6750 4400 6900
+	4400 6750 4400 6800
 Wire Wire Line
 	3650 6250 3700 6250
 Wire Wire Line
-	3650 6050 3650 6800
-Wire Wire Line
-	3650 6800 5200 6800
+	3650 6050 3650 6150
+Wire Wire Line
+	3650 6800 4400 6800
 Connection ~ 4400 6800
 Wire Wire Line
@@
 Connection ~ 3650 6150
 $Comp
-L +V_LOGIC #PWR092
+L RMC:+V_LOGIC #PWR092
 U 1 1 52B2384C
 P 4400 5600
@@
 EEPROM
 $Comp
-L C C601
+L RAMPS-FD-rescue:C C601
 U 1 1 52B22339
 P 6050 6250
@@
 $EndComp
 $Comp
-L GND #PWR094
+L power:GND #PWR094
 U 1 1 52B22346
 P 6050 6600
@@
 	6050 6400 6050 6600
 $Comp
-L +V_LOGIC #PWR094
+L RMC:+V_LOGIC #PWR094
 U 1 1 52B2234D
 P 6050 5900
@@
 Wire Notes Line
 	9250 3550 8450 3550
+Wire Wire Line
+	4800 2400 5450 2400
+Wire Wire Line
+	4450 2500 5450 2500
+Wire Wire Line
+	4800 1650 5250 1650
+Wire Wire Line
+	4450 1650 4450 1850
+Wire Wire Line
+	4450 3850 4450 4050
+Wire Wire Line
+	4800 3850 4450 3850
+Wire Wire Line
+	4450 4700 5450 4700
+Wire Wire Line
+	4800 4600 5450 4600
+Wire Wire Line
+	4400 6800 4400 6900
+Wire Wire Line
+	4400 6800 5200 6800
+Wire Wire Line
+	3650 6250 3650 6800
+Wire Wire Line
+	3650 6150 3650 6250
 $EndSCHEMATC

Commit message: Added UART for Communication with TMC2209 Drivers, improved inverse-polarity protection, added Driver Protection. Two Layer Design
Parts:
- removed K201: S1, Pin_Headers:Pin_Header_Straight_1x03_Pitch2.54mm, symbol RAMPS-FD-rescue:CONN_3
- removed K202: S2, Pin_Headers:Pin_Header_Straight_1x03_Pitch2.54mm, symbol RAMPS-FD-rescue:CONN_3
- removed K203: S3, Pin_Headers:Pin_Header_Straight_1x03_Pitch2.54mm, symbol RAMPS-FD-rescue:CONN_3
- removed K204: S4, Pin_Headers:Pin_Header_Straight_1x03_Pitch2.54mm, symbol RAMPS-FD-rescue:CONN_3
- removed P1: SERIAL1, Pin_Headers:Pin_Header_Straight_1x06_Pitch2.54mm, symbol RAMPS-FD-rescue:CONN_6
- removed P216: SERIAL0, Pin_Headers:Pin_Header_Straight_1x06_Pitch2.54mm, symbol RAMPS-FD-rescue:CONN_6
- removed U601: 24C512, libcms:SO8E, symbol RAMPS-FD-rescue:24C512
- added J17, J20: 1x3PinHeader, RAMPS-FD:PinHeader_1x03_P2.54mm_Vertical, symbol RAMPS-FD:1x3PinHeader
- added J23: 3x4PinHeader, RAMPS-FD:4x3_2.54mm_Header, symbol RAMPS-FD:3x4PinHeader
- added U10: 24C512, RAMPS-FD:SOIC-8_3.9x4.9mm_P1.27mm, symbol RAMPS-FD:24C512
- C12: renamed from C601; footprint Capacitors_SMD:C_0603 -> RAMPS-FD:C_0603; symbol RAMPS-FD-rescue:C -> RAMPS-FD:100n; Fitted (none) -> yes; Ordering (none) -> LCSC: C85999; Price (USD) (none) -> 0,016915; Rating (none) -> #100nF #50V #5%
- J18: renamed from P214; value AUX-2 -> 2x5PinHeader; footprint rmc:PIN_ARRAY_5x2_RMC -> RAMPS-FD:pin_header_2.54mm_2x5; symbol RAMPS-FD-rescue:CONN_5X2 -> RAMPS-FD:2x5PinHeader; Fitted (none) -> yes; Ordering (none) -> LCSC: C124387; Price (USD) (none) -> 0,04557
- J19: renamed from P211; value I2C-0 -> 1x4PinHeader; footprint Pin_Headers:Pin_Header_Straight_1x04_Pitch2.54mm -> RAMPS-FD:pin_header_2.54mm_1x4; symbol RAMPS-FD-rescue:CONN_4 -> RAMPS-FD:1x4PinHeader; Fitted (none) -> yes; Ordering (none) -> LCSC: C124378; Price (USD) (none) -> 0,024235
- J21: renamed from P215; value AUX-3 -> 2x6PinHeader; footprint rmc:PIN_ARRAY_6x2_RMC -> RAMPS-FD:pin_header_2.54mm_2x6; symbol RAMPS-FD-rescue:CONN_6X2 -> RAMPS-FD:2x6PinHeader; Fitted (none) -> yes; Ordering (none) -> LCSC: C124388; Price (USD) (none) -> 0,057859
- J22: renamed from P2; value I2C-1 -> 1x4PinHeader; footprint Pin_Headers:Pin_Header_Straight_1x04_Pitch2.54mm -> RAMPS-FD:pin_header_2.54mm_1x4; symbol RAMPS-FD-rescue:CONN_4 -> RAMPS-FD:1x4PinHeader; Fitted (none) -> yes; Ordering (none) -> LCSC: C124378; Price (USD) (none) -> 0,024235
- J24: renamed from P213; value AUX-4 -> 1x18PinHeader; footprint Pin_Headers:Pin_Header_Straight_1x18_Pitch2.54mm -> RAMPS-FD:PinHeader_1x18_P2.54mm_Vertical; symbol RMC:CONN_18 -> RAMPS-FD:1x18PinHeader; Fitted (none) -> yes; Ordering (none) -> LCSC: 1xC124381 1xC124372; Price (USD) (none) -> =0,047589+0,048216
- R22: renamed from R211; value NF -> 10k; footprint Resistors_SMD:R_0603 -> RAMPS-FD:R_0603; symbol RAMPS-FD-rescue:R -> RAMPS-FD:10k; Fitted (none) -> yes; Ordering (none) -> LCSC: C238881; Price (USD) (none) -> 0,003395
- R23: renamed from R212; value NF -> 10k; footprint Resistors_SMD:R_0603 -> RAMPS-FD:R_0603; symbol RAMPS-FD-rescue:R -> RAMPS-FD:10k; Fitted (none) -> yes; Ordering (none) -> LCSC: C238881; Price (USD) (none) -> 0,003395
- R24: renamed from R1; value NF -> 10k; footprint Resistors_SMD:R_0603 -> RAMPS-FD:R_0603; symbol RAMPS-FD-rescue:R -> RAMPS-FD:10k; Fitted (none) -> yes; Ordering (none) -> LCSC: C238881; Price (USD) (none) -> 0,003395
- R25: renamed from R2; value NF -> 10k; footprint Resistors_SMD:R_0603 -> RAMPS-FD:R_0603; symbol RAMPS-FD-rescue:R -> RAMPS-FD:10k; Fitted (none) -> yes; Ordering (none) -> LCSC: C238881; Price (USD) (none) -> 0,003395
Connections:
- wire segments 120 -> 125
- no-connect marks 7 -> 1
Other:
- note removed: "Need buffered outputs?"
