File: RAMPS-FD/con_outputs.sch (KiCad schematic (older format))
At the start: 24 parts, among them P218 D11, P403 D9, P404 D8, P405 D10, Q201 IRLB8743PBF, Q202 IRLB8743PBF, Q203 IRLB8743PBF, Q206 IRLB8743PBF

Commit message: Inital Commit RAMPS FD v2.3. SPI Support for every Driver added.
Parts:
- D201, D202, D203, D204: symbol LED-RESCUE-RAMPS-FD -> RAMPS-FD-rescue:LED-RESCUE-RAMPS-FD
- D401, D402, D403, D404: symbol D -> RAMPS-FD-rescue:D
- P218, P403, P404, P405: symbol CONN_2 -> RAMPS-FD-rescue:CONN_2
- Q201, Q202, Q203, Q206: symbol MOSFET_N_RMC -> RMC:MOSFET_N_RMC
- R219, R220, R221, R222, R701, R702, R703, R704: symbol R -> RAMPS-FD-rescue:R
Changed lines of the file:
@@
-EESchema Schematic File Version 2
-LIBS:RAMPS-FD-rescue
-LIBS:power
-LIBS:device
-LIBS:transistors
-LIBS:conn
-LIBS:linear
-LIBS:regul
-LIBS:74xx
-LIBS:cmos4000
-LIBS:adc-dac
-LIBS:memory
-LIBS:xilinx
-LIBS:microcontrollers
-LIBS:dsp
-LIBS:microchip
-LIBS:analog_switches
-LIBS:motorola
-LIBS:texas
-LIBS:intel
-LIBS:audio
-LIBS:interface
-LIBS:digital-audio
-LIBS:philips
-LIBS:display
-LIBS:cypress
-LIBS:siliconi
-LIBS:opto
-LIBS:atmel
-LIBS:contrib
-LIBS:valves
-LIBS:RMC
-LIBS:RAMPS-FD-cache
-EELAYER 25 0
+EESchema Schematic File Version 4
+EELAYER 30 0
 EELAYER END
 $Descr A4 11693 8268
@@
 Sheet 7 10
 Title "RAMPS-FD (RAMPS for Arduino Due)"
-Date "2016-07-17"
-Rev "v2.2"
+Date "2019-04-13"
+Rev "v2.3"
 Comp ""
-Comment1 "Derived from RAMPS 1.4 reprap.org/wiki/RAMPS1.4"
+Comment1 "Derived from RAMPS FD 2.2 by Bob Cousins github.com/bobc/bobc_hardware/"
 Comment2 "GPL v3"
-Comment3 "Bob Cousins 2016"
+Comment3 "Marius Krause 2019"
 Comment4 ""
 $EndDescr
@@
 D8 - Heatbed
 $Comp
-L GNDPWR #PWR095
+L RAMPS-FD-rescue:GNDPWR #PWR095
 U 1 1 51AA07E6
 P 9300 3000
@@
 $EndComp
 $Comp
-L GNDPWR #PWR096
+L RAMPS-FD-rescue:GNDPWR #PWR096
 U 1 1 51AA0719
 P 9450 6350
@@
 $EndComp
 $Comp
-L GNDPWR #PWR097
+L RAMPS-FD-rescue:GNDPWR #PWR097
 U 1 1 51AA06B9
 P 3350 6550
@@
 $EndComp
 $Comp
-L CONN_2 P405
+L RAMPS-FD-rescue:CONN_2 P405
 U 1 1 51AA03B1
 P 10600 5300
@@
 $EndComp
 $Comp
-L CONN_2 P403
+L RAMPS-FD-rescue:CONN_2 P403
 U 1 1 51AA03AE
 P 4700 5250
@@
 $EndComp
 $Comp
-L CONN_2 P404
+L RAMPS-FD-rescue:CONN_2 P404
 U 1 1 51AA03A7
 P 4850 1950
@@
 $EndComp
 $Comp
-L D D404
+L RAMPS-FD-rescue:D D404
 U 1 1 51A9D334
 P 3650 1500
@@
 $EndComp
 $Comp
-L D D403
+L RAMPS-FD-rescue:D D403
 U 1 1 519E92CD
 P 9600 1400
@@
 $EndComp
 $Comp
-L D D401
+L RAMPS-FD-rescue:D D401
 U 1 1 519E9216
 P 3350 4800
@@
 $EndComp
 $Comp
-L D D402
+L RAMPS-FD-rescue:D D402
 U 1 1 5186017E
 P 9450 4850
@@
 $EndComp
 $Comp
-L CONN_2 P218
+L RAMPS-FD-rescue:CONN_2 P218
 U 1 1 51770F88
 P 10700 1850
@@
 $EndComp
 $Comp
-L LED-RESCUE-RAMPS-FD D204
+L RAMPS-FD-rescue:LED-RESCUE-RAMPS-FD D204
 U 1 1 51770EF9
 P 8900 1700
@@
 $EndComp
 $Comp
-L R R222
+L RAMPS-FD-rescue:R R222
 U 1 1 51770EF8
 P 8900 1150
@@
 FET4_BUF
 $Comp
-L MOSFET_N_RMC Q206
+L RMC:MOSFET_N_RMC Q206
 U 1 1 51770EF3
 P 9250 2250
@@
 $EndComp
 $Comp
-L +V_POWER #PWR098
+L RMC:+V_POWER #PWR098
 U 1 1 51770EF2
 P 9600 650
@@
 FET4_OUT
 $Comp
-L MOSFET_N_RMC Q201
+L RMC:MOSFET_N_RMC Q201
 U 1 1 510E6DBE
 P 3250 2450
@@
 D8_OUT
 $Comp
-L +V_POWER #PWR099
+L RMC:+V_POWER #PWR099
 U 1 1 5176EF23
 P 3350 4150
@@
 $EndComp
 $Comp
-L +V_POWER #PWR0100
+L RMC:+V_POWER #PWR0100
 U 1 1 5176EE9D
 P 9450 4050
@@
 $EndComp
 $Comp
-L +V_HEATBED #PWR0101
+L RMC:+V_HEATBED #PWR0101
 U 1 1 5176EDD7
 P 3650 700
@@
 $EndComp
 $Comp
-L MOSFET_N_RMC Q203
+L RMC:MOSFET_N_RMC Q203
 U 1 1 510E6E63
 P 3300 5750
@@
 $EndComp
 $Comp
-L MOSFET_N_RMC Q202
+L RMC:MOSFET_N_RMC Q202
 U 1 1 510E6E60
 P 9400 5700
@@
 MOSFET Outputs
 $Comp
-L LED-RESCUE-RAMPS-FD D203
+L RAMPS-FD-rescue:LED-RESCUE-RAMPS-FD D203
 U 1 1 51047AB7
 P 2850 5100
@@
 $EndComp
 $Comp
-L R R221
+L RAMPS-FD-rescue:R R221
 U 1 1 51047AB6
 P 2850 4600
@@
 D9_BUF
 $Comp
-L R R220
+L RAMPS-FD-rescue:R R220
 U 1 1 510479AF
 P 9000 4600
@@
 $EndComp
 $Comp
-L LED-RESCUE-RAMPS-FD D202
+L RAMPS-FD-rescue:LED-RESCUE-RAMPS-FD D202
 U 1 1 510479AE
 P 9000 5150
@@
 $EndComp
 $Comp
-L LED-RESCUE-RAMPS-FD D201
+L RAMPS-FD-rescue:LED-RESCUE-RAMPS-FD D201
 U 1 1 510478C6
 P 2700 1800
@@
 $EndComp
 $Comp
-L R R219
+L RAMPS-FD-rescue:R R219
 U 1 1 510478C3
 P 2700 1250
@@
 	1100 5800 1700 5800
 $Comp
-L GNDPWR #PWR0102
+L RAMPS-FD-rescue:GNDPWR #PWR0102
 U 1 1 5251556C
 P 3300 3050
@@
 $EndComp
 $Comp
-L R R701
+L RAMPS-FD-rescue:R R701
 U 1 1 52B221FB
 P 1800 2500
@@
 	1050 2500 1650 2500
 $Comp
-L R R702
+L RAMPS-FD-rescue:R R702
 U 1 1 52B22B4E
 P 1850 5800
@@
 $EndComp
 $Comp
-L R R704
+L RAMPS-FD-rescue:R R704
 U 1 1 52B22CEA
 P 8050 5750
@@
 $EndComp
 $Comp
-L R R703
+L RAMPS-FD-rescue:R R703
 U 1 1 52B22C21
 P 7950 2300

Commit message: Added UART for Communication with TMC2209 Drivers, improved inverse-polarity protection, added Driver Protection. Two Layer Design
Parts:
- D20: renamed from D403; value ES1F -> MRA4003T3G; footprint rmc:DO-214AC -> RAMPS-FD:D_SMA; symbol RAMPS-FD-rescue:D -> RAMPS-FD:MRA4003T3G; Fitted (none) -> yes; Ordering (none) -> LCSC: C94410; Price (USD) (none) -> 0,049228; Rating (none) -> #300V #1A
- D21: renamed from D404; value ES1F -> MRA4003T3G; footprint rmc:DO-214AC -> RAMPS-FD:D_SMA; symbol RAMPS-FD-rescue:D -> RAMPS-FD:MRA4003T3G; Fitted (none) -> yes; Ordering (none) -> LCSC: C94410; Price (USD) (none) -> 0,049228; Rating (none) -> #300V #1A
- D22: renamed from D204; value LED RED -> LED_0603_RED; footprint rmc:LED-0805_RED -> RAMPS-FD:LED_0603; symbol RAMPS-FD-rescue:LED-RESCUE-RAMPS-FD -> RAMPS-FD:LED_0603_RED; Fitted (none) -> yes; Ordering (none) -> LCSC: C192315; Price (USD) (none) -> 0,018284
- D23: renamed from D201; value LED RED -> LED_0603_RED; footprint rmc:LED-0805_RED -> RAMPS-FD:LED_0603; symbol RAMPS-FD-rescue:LED-RESCUE-RAMPS-FD -> RAMPS-FD:LED_0603_RED; Fitted (none) -> yes; Ordering (none) -> LCSC: C192315; Price (USD) (none) -> 0,018284
- D24: renamed from D401; value ES1F -> MRA4003T3G; footprint rmc:DO-214AC -> RAMPS-FD:D_SMA; symbol RAMPS-FD-rescue:D -> RAMPS-FD:MRA4003T3G; Fitted (none) -> yes; Ordering (none) -> LCSC: C94410; Price (USD) (none) -> 0,049228; Rating (none) -> #300V #1A
- D25: renamed from D402; value ES1F -> MRA4003T3G; footprint rmc:DO-214AC -> RAMPS-FD:D_SMA; symbol RAMPS-FD-rescue:D -> RAMPS-FD:MRA4003T3G; Fitted (none) -> yes; Ordering (none) -> LCSC: C94410; Price (USD) (none) -> 0,049228; Rating (none) -> #300V #1A
- D26: renamed from D203; value LED RED -> LED_0603_RED; footprint rmc:LED-0805_RED -> RAMPS-FD:LED_0603; symbol RAMPS-FD-rescue:LED-RESCUE-RAMPS-FD -> RAMPS-FD:LED_0603_RED; Fitted (none) -> yes; Ordering (none) -> LCSC: C192315; Price (USD) (none) -> 0,018284
- D27: renamed from D202; value LED RED -> LED_0603_RED; footprint rmc:LED-0805_RED -> RAMPS-FD:LED_0603; symbol RAMPS-FD-rescue:LED-RESCUE-RAMPS-FD -> RAMPS-FD:LED_0603_RED; Fitted (none) -> yes; Ordering (none) -> LCSC: C192315; Price (USD) (none) -> 0,018284
- J25: renamed from P218; value D11 -> 2_PinScrewTerminal_P350; footprint rmc:RMC-pt_1,5-2-3,5-h -> RAMPS-FD:2x1_P350; symbol RAMPS-FD-rescue:CONN_2 -> RAMPS-FD:2_PinScrewTerminal_P350; Fitted (none) -> yes; Ordering (none) -> LCSC: C474892; Price (USD) (none) -> 0,07
- J26: renamed from P404; value D8 -> 2_PinScrewTerminal_P508; footprint w_conn_screw:mors_2p -> RAMPS-FD:2x1_P508; symbol RAMPS-FD-rescue:CONN_2 -> RAMPS-FD:2_PinScrewTerminal_P508; Fitted (none) -> yes; Ordering (none) -> LCSC: C474952; Price (USD) (none) -> 0,13895
- J27: renamed from P403; value D9 -> 2_PinScrewTerminal_P350; footprint rmc:RMC-pt_1,5-2-3,5-h -> RAMPS-FD:2x1_P350; symbol RAMPS-FD-rescue:CONN_2 -> RAMPS-FD:2_PinScrewTerminal_P350; Fitted (none) -> yes; Ordering (none) -> LCSC: C474892; Price (USD) (none) -> 0,07
- J28: renamed from P405; value D10 -> 2_PinScrewTerminal_P350; footprint rmc:RMC-pt_1,5-2-3,5-h -> RAMPS-FD:2x1_P350; symbol RAMPS-FD-rescue:CONN_2 -> RAMPS-FD:2_PinScrewTerminal_P350; Fitted (none) -> yes; Ordering (none) -> LCSC: C474892; Price (USD) (none) -> 0,07
- Q6: renamed from Q206; value IRLB8743PBF -> PSMN7R5-60YLX; footprint rmc:TO-220AB_IRF2804_RMC -> RAMPS-FD:LFPAK56; symbol RMC:MOSFET_N_RMC -> RAMPS-FD:PSMN7R5-60YLX; Fitted (none) -> yes; Ordering (none) -> LCSC: C478175; Price (USD) (none) -> 0,972045; Rating (none) -> #60V #86A
- Q7: renamed from Q201; value IRLB8743PBF -> PSMN1R8-40YLC; footprint rmc:TO-220AB_IRF2804_RMC -> RAMPS-FD:LFPAK56; symbol RMC:MOSFET_N_RMC -> RAMPS-FD:PSMN1R8-40YLC; Fitted (none) -> yes; Ordering (none) -> LCSC: C124522; Price (USD) (none) -> 0,281273; Rating (none) -> #40V #100A
- Q8: renamed from Q202; value IRLB8743PBF -> PSMN7R5-60YLX; footprint rmc:TO-220AB_IRF2804_RMC -> RAMPS-FD:LFPAK56; symbol RMC:MOSFET_N_RMC -> RAMPS-FD:PSMN7R5-60YLX; Fitted (none) -> yes; Ordering (none) -> LCSC: C478175; Price (USD) (none) -> 0,972045; Rating (none) -> #60V #86A
- Q9: renamed from Q203; value IRLB8743PBF -> PSMN7R5-60YLX; footprint rmc:TO-220AB_IRF2804_RMC -> RAMPS-FD:LFPAK56; symbol RMC:MOSFET_N_RMC -> RAMPS-FD:PSMN7R5-60YLX; Fitted (none) -> yes; Ordering (none) -> LCSC: C478175; Price (USD) (none) -> 0,972045; Rating (none) -> #60V #86A
- R26: renamed from R222; footprint Resistors_SMD:R_0603 -> RAMPS-FD:R_0603; symbol RAMPS-FD-rescue:R -> RAMPS-FD:1k; Fitted (none) -> yes; Ordering (none) -> LCSC: C328340; Price (USD) (none) -> 0,003087
- R27: renamed from R219; footprint Resistors_SMD:R_0603 -> RAMPS-FD:R_0603; symbol RAMPS-FD-rescue:R -> RAMPS-FD:1k; Fitted (none) -> yes; Ordering (none) -> LCSC: C328340; Price (USD) (none) -> 0,003087
- R28: renamed from R703; value 220R -> 33R; footprint Resistors_SMD:R_0603 -> RAMPS-FD:R_0603; symbol RAMPS-FD-rescue:R -> RAMPS-FD:33R; Fitted (none) -> yes; Ordering (none) -> LCSC: C325638; Price (USD) (none) -> 0,002066
- R29: renamed from R701; value 220R -> 33R; footprint Resistors_SMD:R_0603 -> RAMPS-FD:R_0603; symbol RAMPS-FD-rescue:R -> RAMPS-FD:33R; Fitted (none) -> yes; Ordering (none) -> LCSC: C325638; Price (USD) (none) -> 0,002066
- R30: renamed from R221; footprint Resistors_SMD:R_0603 -> RAMPS-FD:R_0603; symbol RAMPS-FD-rescue:R -> RAMPS-FD:1k; Fitted (none) -> yes; Ordering (none) -> LCSC: C328340; Price (USD) (none) -> 0,003087
- R31: renamed from R220; footprint Resistors_SMD:R_0603 -> RAMPS-FD:R_0603; symbol RAMPS-FD-rescue:R -> RAMPS-FD:1k; Fitted (none) -> yes; Ordering (none) -> LCSC: C328340; Price (USD) (none) -> 0,003087
- R32: renamed from R704; value 220R -> 33R; footprint Resistors_SMD:R_0603 -> RAMPS-FD:R_0603; symbol RAMPS-FD-rescue:R -> RAMPS-FD:33R; Fitted (none) -> yes; Ordering (none) -> LCSC: C325638; Price (USD) (none) -> 0,002066
- R33: renamed from R702; value 220R -> 33R; footprint Resistors_SMD:R_0603 -> RAMPS-FD:R_0603; symbol RAMPS-FD-rescue:R -> RAMPS-FD:33R; Fitted (none) -> yes; Ordering (none) -> LCSC: C325638; Price (USD) (none) -> 0,002066
Connections:
- wire segments 50 -> 72
