File: RAMPS-FD/e-stop.sch (KiCad schematic (older format))
At the start: 17 parts, among them P302 ESTOP, Q1 DMN2075, U1 74HCT125, U2 74HCT244

Commit message: Inital Commit RAMPS FD v2.3. SPI Support for every Driver added.
Parts:
- C1, C2: symbol C -> RAMPS-FD-rescue:C
- D1: symbol LED-RESCUE-RAMPS-FD -> RAMPS-FD-rescue:LED-RESCUE-RAMPS-FD
- D301: symbol D -> RAMPS-FD-rescue:D
- P302: symbol CONN_2 -> RAMPS-FD-rescue:CONN_2
- Q1: symbol MOSFET_N -> RMC:MOSFET_N
- R3, R304, R305, R401, R402: symbol R -> RAMPS-FD-rescue:R
- RP1, RP2, RP3, RP401: symbol R_PACK4 -> RAMPS-FD-rescue:R_PACK4
- U1: symbol 74LS125 -> RAMPS-FD-rescue:74LS125
- U2: symbol 74LS244 -> RAMPS-FD-rescue:74LS244
Changed lines of the file:
@@
-EESchema Schematic File Version 2
-LIBS:RAMPS-FD-rescue
-LIBS:power
-LIBS:device
-LIBS:transistors
-LIBS:conn
-LIBS:linear
-LIBS:regul
-LIBS:74xx
-LIBS:cmos4000
-LIBS:adc-dac
-LIBS:memory
-LIBS:xilinx
-LIBS:microcontrollers
-LIBS:dsp
-LIBS:microchip
-LIBS:analog_switches
-LIBS:motorola
-LIBS:texas
-LIBS:intel
-LIBS:audio
-LIBS:interface
-LIBS:digital-audio
-LIBS:philips
-LIBS:display
-LIBS:cypress
-LIBS:siliconi
-LIBS:opto
-LIBS:atmel
-LIBS:contrib
-LIBS:valves
-LIBS:RMC
-LIBS:RAMPS-FD-cache
-EELAYER 25 0
+EESchema Schematic File Version 4
+EELAYER 30 0
 EELAYER END
 $Descr A4 11693 8268
@@
 Sheet 4 10
 Title "RAMPS-FD (RAMPS for Arduino Due)"
-Date "2016-07-17"
-Rev "v2.2"
+Date "2019-04-13"
+Rev "v2.3"
 Comp ""
-Comment1 "Derived from RAMPS 1.4 reprap.org/wiki/RAMPS1.4"
+Comment1 "Derived from RAMPS FD 2.2 by Bob Cousins github.com/bobc/bobc_hardware/"
 Comment2 "GPL v3"
-Comment3 "Bob Cousins 2016"
+Comment3 "Marius Krause 2019"
 Comment4 ""
 $EndDescr
 $Comp
-L VCC #PWR045
+L power:VCC #PWR045
 U 1 1 523A3B4A
 P 6200 1200
@@
 $EndComp
 $Comp
-L R_PACK4 RP1
+L RAMPS-FD-rescue:R_PACK4 RP1
 U 1 1 523A3B30
 P 6450 6900
@@
 $EndComp
 $Comp
-L R_PACK4 RP3
+L RAMPS-FD-rescue:R_PACK4 RP3
 U 1 1 523A3B2E
 P 7250 1700
@@
 $EndComp
 $Comp
-L R_PACK4 RP2
+L RAMPS-FD-rescue:R_PACK4 RP2
 U 1 1 523A3B27
 P 6550 1700
@@
 D10_BUF
 $Comp
-L GND #PWR049
+L power:GND #PWR049
 U 1 1 523A374A
 P 3700 7600
@@
 D10
 $Comp
-L 74LS125 U1
+L RAMPS-FD-rescue:74LS125 U1
 U 1 1 523A36ED
 P 4850 6450
@@
 $EndComp
 $Comp
-L 74LS125 U1
+L RAMPS-FD-rescue:74LS125 U1
 U 4 1 523A36EC
 P 4900 5700
@@
 $EndComp
 $Comp
-L 74LS125 U1
+L RAMPS-FD-rescue:74LS125 U1
 U 3 1 523A36E7
 P 4900 5100
@@
 $EndComp
 $Comp
-L 74LS125 U1
+L RAMPS-FD-rescue:74LS125 U1
 U 2 1 523A36E3
 P 4900 4350
@@
 $EndComp
 $Comp
-L 74LS244 U2
+L RAMPS-FD-rescue:74LS244 U2
 U 1 1 523A33CC
 P 5100 2800
@@
 $EndComp
 $Comp
-L VCC #PWR047
+L power:VCC #PWR047
 U 1 1 51E4F650
 P 10650 900
@@
 $EndComp
 $Comp
-L GND #PWR051
+L power:GND #PWR051
 U 1 1 51E4F64F
 P 10650 1700
@@
 $EndComp
 $Comp
-L C C2
+L RAMPS-FD-rescue:C C2
 U 1 1 51E4F64E
 P 10650 1300
@@
 $EndComp
 $Comp
-L C C1
+L RAMPS-FD-rescue:C C1
 U 1 1 51E4F640
 P 10100 1300
@@
 $EndComp
 $Comp
-L GND #PWR052
+L power:GND #PWR052
 U 1 1 51E4F630
 P 10100 1700
@@
 $EndComp
 $Comp
-L VCC #PWR050
+L power:VCC #PWR050
 U 1 1 51E4F62B
 P 10100 900
@@
 D8
 $Comp
-L D D301
+L RAMPS-FD-rescue:D D301
 U 1 1 51B65AB0
 P 1900 1600
@@
 $EndComp
 $Comp
-L R R305
+L RAMPS-FD-rescue:R R305
 U 1 1 51B4ECD2
 P 1300 2050
@@
 $EndComp
 $Comp
-L +V_LOGIC #PWR051
+L RMC:+V_LOGIC #PWR051
 U 1 1 51B4EC55
 P 1550 1000
@@
 $EndComp
 $Comp
-L CONN_2 P302
+L RAMPS-FD-rescue:CONN_2 P302
 U 1 1 51B4EBF7
 P 800 1700
@@
 $EndComp
 $Comp
-L R R304
+L RAMPS-FD-rescue:R R304
 U 1 1 51B4EBD5
 P 1550 1250
@@
 $EndComp
 $Comp
-L GND #PWR055
+L power:GND #PWR055
 U 1 1 51B4EBC7
 P 1300 2350
@@
 Active high
 $Comp
-L R R401
+L RAMPS-FD-rescue:R R401
 U 1 1 52B0D0FC
 P 3400 3650
@@
 $EndComp
 $Comp
-L R R402
+L RAMPS-FD-rescue:R R402
 U 1 1 52B0D109
 P 3700 3650
@@
 $EndComp
 $Comp
-L GND #PWR056
+L power:GND #PWR056
 U 1 1 52B0D127
 P 3700 4150
@@
 $EndComp
 $Comp
-L GND #PWR057
+L power:GND #PWR057
 U 1 1 52B224D5
 P 7500 1550
@@
 $EndComp
 $Comp
-L R_PACK4 RP401
+L RAMPS-FD-rescue:R_PACK4 RP401
 U 1 1 52B22857
 P 3850 6950
@@
 $EndComp
 $Comp
-L GND #PWR058
+L power:GND #PWR058
 U 1 1 52B22A39
 P 6300 7550
@@
 	825  1450 825  775
 $Comp
-L LED-RESCUE-RAMPS-FD D1
+L RAMPS-FD-rescue:LED-RESCUE-RAMPS-FD D1
 U 1 1 5725588E
 P 1450 4850
@@
 $EndComp
 $Comp
-L GND #PWR056
+L power:GND #PWR056
 U 1 1 572566C5
 P 1450 5775
@@
 $EndComp
 $Comp
-L R R3
+L RAMPS-FD-rescue:R R3
 U 1 1 572566D2
 P 1450 4425
@@
 $EndComp
 $Comp
-L +5V #PWR057
+L power:+5V #PWR057
 U 1 1 572566D9
 P 1450 4200
@@
 $EndComp
 $Comp
-L MOSFET_N Q1
+L RMC:MOSFET_N Q1
 U 1 1 572566DF
 P 1375 5425

Commit message: Added UART for Communication with TMC2209 Drivers, improved inverse-polarity protection, added Driver Protection. Two Layer Design
Parts:
- removed C2: 100n, Capacitors_SMD:C_0603, symbol RAMPS-FD-rescue:C
- removed R3: 330R, Resistors_SMD:R_0603, symbol RAMPS-FD-rescue:R
- removed R401, R402: 10k, Resistors_SMD:R_0603, symbol RAMPS-FD-rescue:R
- removed RP1: 10k, Resistors_SMD:R_Cat16-4, symbol RAMPS-FD-rescue:R_PACK4
- removed U1: 74HCT125, Housings_SSOP:TSSOP-14_4.4x5mm_Pitch0.65mm, symbol RAMPS-FD-rescue:74LS125
- removed U2: 74HCT244, Housings_SSOP:TSSOP-20_4.4x6.5mm_Pitch0.65mm, symbol RAMPS-FD-rescue:74LS244
- added R14: 330R, RAMPS-FD:R_0603, symbol RAMPS-FD:330R
- added U6: SN74LV1T125, RAMPS-FD:SOT-23-5, symbol RAMPS-FD:SN74LV1T125
- C8: renamed from C1; footprint Capacitors_SMD:C_0603 -> RAMPS-FD:C_0603; symbol RAMPS-FD-rescue:C -> RAMPS-FD:100n; Fitted (none) -> yes; Ordering (none) -> LCSC: C85999; Price (USD) (none) -> 0,016915; Rating (none) -> #100nF #50V #5%
- D12: renamed from D301; value 1N4148 -> 2CZ4007; footprint Diodes_SMD:SOD-123 -> RAMPS-FD:D_SOD-123F; symbol RAMPS-FD-rescue:D -> RAMPS-FD:2CZ4007; Fitted (none) -> yes; Ordering (none) -> LCSC: C85712; Price (USD) (none) -> 0,05; Rating (none) -> #1kV #1A
- D13: renamed from D1; value ESTOP -> LED_0603_GREEN; footprint rmc:LED-0805_GREEN -> RAMPS-FD:LED_0603; symbol RAMPS-FD-rescue:LED-RESCUE-RAMPS-FD -> RAMPS-FD:LED_0603_GREEN; Fitted (none) -> yes; Ordering (none) -> LCSC: C192316; Price (USD) (none) -> 0,021656
- J13: renamed from P302; value ESTOP -> 2x1PinHeader; footprint rmc:CONN_KK_2.54_2W -> RAMPS-FD:PinHeader_1x02_P2.54mm_Vertical; symbol RAMPS-FD-rescue:CONN_2 -> RAMPS-FD:2x1PinHeader; Fitted (none) -> yes; Ordering (none) -> LCSC: C124375; Price (USD) (none) -> 0,015147
- Q5: renamed from Q1; value DMN2075 -> NCE3416; footprint libcms:SOT23GDS -> RAMPS-FD:SOT-23; symbol RMC:MOSFET_N -> RAMPS-FD:NCE3416; Fitted (none) -> yes; Ordering (none) -> LCSC: C113491; Price (USD) (none) -> 0,033091; Rating (none) -> #20V #6.5A
- R12: renamed from R304; footprint Resistors_SMD:R_0603 -> RAMPS-FD:R_0603; symbol RAMPS-FD-rescue:R -> RAMPS-FD:100k; Fitted (none) -> yes; Ordering (none) -> LCSC: C237792; Price (USD) (none) -> 0,003527
- R13: renamed from R305; footprint Resistors_SMD:R_0603 -> RAMPS-FD:R_0603; symbol RAMPS-FD-rescue:R -> RAMPS-FD:4k7; Fitted (none) -> yes; Ordering (none) -> LCSC: C137710; Price (USD) (none) -> 0,002446
- RP2, RP3: value 10k -> 10kArrayx4; footprint Resistors_SMD:R_Cat16-4 -> RAMPS-FD:R_Array_Convex_4x0603; symbol RAMPS-FD-rescue:R_PACK4 -> RAMPS-FD:10kArrayx4; Fitted (none) -> yes; Ordering (none) -> LCSC: C29718; Price (USD) (none) -> 0,007304
- RP4: renamed from RP401; value 10k -> 10kArrayx4; footprint Resistors_SMD:R_Cat16-4 -> RAMPS-FD:R_Array_Convex_4x0603; symbol RAMPS-FD-rescue:R_PACK4 -> RAMPS-FD:10kArrayx4; Fitted (none) -> yes; Ordering (none) -> LCSC: C29718; Price (USD) (none) -> 0,007304
Connections:
- net labels removed: VCC
- wire segments 90 -> 89
Other:
- note added: "Use a Buffer to translate the 3V3 Signal of the Due to 5V to fully open the Mosfet\nPossible alternative parts (pin compatible):\n74LVC1G17\nSN74LV1T34\n"
- note removed: "Must use HCT type buffers. \nInputs are compatible with \n3.3V or 5V logic"
- note removed: "VCC = 5V"
