File: RAMPS-FD/steppers.sch (KiCad schematic (older format))
At the start: 25 parts, among them J3 CONN_02X03, J4 CONN_02X03, J5 CONN_02X03, P201 3 2 1, P202 3 2 1, P203 3 2 1, P204 X, P205 Y, P206 Z1, P3 Z2, U201 X, U202 Y, U203 Z

Commit message: Inital Commit RAMPS FD v2.3. SPI Support for every Driver added.
Parts:
- removed J3, J4, J5: CONN_02X03, Pin_Headers:Pin_Header_Straight_2x03_Pitch2.54mm, symbol CONN_02X03
- removed P201, P202, P203: 3 2 1, Pin_Headers:Pin_Header_Straight_2x03_Pitch2.54mm, symbol CONN_3X2
- removed R5, R8, R9: 10k, Resistors_SMD:R_0603, symbol R
- added P4, P5, P6: SPI Selector, Connector_PinHeader_2.54mm:PinHeader_2x04_P2.54mm_Vertical, symbol RAMPS-FD-rescue:CONN_4X2
- added P7, P8, P9: Pullup Sel., Connector_PinHeader_2.54mm:PinHeader_1x04_P2.54mm_Vertical, symbol RAMPS-FD-rescue:CONN_4
- C201, C202, C203: symbol CP1 -> RAMPS-FD-rescue:CP1
- P204, P205, P206, P3: symbol CONN_4 -> RAMPS-FD-rescue:CONN_4
- R201, R202, R203, R4, R6, R7: symbol R -> RAMPS-FD-rescue:R
- U201, U202, U203: symbol POLOLU -> RMC:POLOLU
Connections:
- wire segments 118 -> 135
Other:
- note added: "Use Jumpers to Connect the SPI Bus to your Stepperdrivers, \nfor example for TMC 2130, \nor to select the microstepping for your Pololu by connecting \nthe middle pin row to +V_Logic"
- moved on the sheet: C203, P206, P3, R201, R7

Commit message: Added UART for Communication with TMC2209 Drivers, improved inverse-polarity protection, added Driver Protection. Two Layer Design
Parts:
- removed P4, P5, P6: SPI Selector, Connector_PinHeader_2.54mm:PinHeader_2x04_P2.54mm_Vertical, symbol RAMPS-FD-rescue:CONN_4X2
- removed P7, P8, P9: Pullup Sel., Connector_PinHeader_2.54mm:PinHeader_1x04_P2.54mm_Vertical, symbol RAMPS-FD-rescue:CONN_4
- added D10, D6, D8: DS110W, RAMPS-FD:D_SOD-123F, symbol RAMPS-FD:DS110W
- added D11, D7, D9: SMF36CA, RAMPS-FD:D_SOD-123F, symbol RAMPS-FD:SMF36CA
- added JP4, JP6, JP8: 4x3JumperArray, RAMPS-FD:4x3_2.54mm_Header, symbol RAMPS-FD:4x3JumperArray
- added JP5, JP7, JP9: 1x2JumperArray, RAMPS-FD:PinHeader_1x02_P2.54mm_Vertical, symbol RAMPS-FD:1x2JumperArray
- added R5: 1k, RAMPS-FD:R_0603, symbol RAMPS-FD:1k
- added VR10, VR11, VR12, VR13, VR14, VR15, VR16, VR17, VR18, VR19, VR2, VR3, VR4, VR5, VR6, VR7, VR8, VR9: 33V, RAMPS-FD:R_0603, symbol RAMPS-FD:33V
- C5: renamed from C201; value 100u 35V -> 100u_35V; footprint Capacitors_SMD:CP_Elec_6.3x7.7 -> RAMPS-FD:CP_Elec_6.3x7.7; symbol RAMPS-FD-rescue:CP1 -> RAMPS-FD:100u_35V; Fitted (none) -> yes; Ordering (none) -> LCSC: C88675; Price (USD) (none) -> 0,067122; Rating (none) -> #100uF #35V #20%
- C6: renamed from C202; value 100u 35V -> 100u_35V; footprint Capacitors_SMD:CP_Elec_6.3x7.7 -> RAMPS-FD:CP_Elec_6.3x7.7; symbol RAMPS-FD-rescue:CP1 -> RAMPS-FD:100u_35V; Fitted (none) -> yes; Ordering (none) -> LCSC: C88675; Price (USD) (none) -> 0,067122; Rating (none) -> #100uF #35V #20%
- C7: renamed from C203; value 100u 35V -> 100u_35V; footprint Capacitors_SMD:CP_Elec_6.3x7.7 -> RAMPS-FD:CP_Elec_6.3x7.7; symbol RAMPS-FD-rescue:CP1 -> RAMPS-FD:100u_35V; Fitted (none) -> yes; Ordering (none) -> LCSC: C88675; Price (USD) (none) -> 0,067122; Rating (none) -> #100uF #35V #20%
- J10: renamed from P205; value Y -> 1x4PinHeader; footprint rmc:CONN_KK_2.54_4W -> RAMPS-FD:pin_header_2.54mm_1x4; symbol RAMPS-FD-rescue:CONN_4 -> RAMPS-FD:1x4PinHeader; Fitted (none) -> yes; Ordering (none) -> LCSC: C124378; Price (USD) (none) -> 0,024235
- J11: renamed from P206; value Z1 -> 1x4PinHeader; footprint rmc:CONN_KK_2.54_4W -> RAMPS-FD:pin_header_2.54mm_1x4; symbol RAMPS-FD-rescue:CONN_4 -> RAMPS-FD:1x4PinHeader; Fitted (none) -> yes; Ordering (none) -> LCSC: C124378; Price (USD) (none) -> 0,024235
- J12: renamed from P3; value Z2 -> 1x4PinHeader; footprint rmc:CONN_KK_2.54_4W -> RAMPS-FD:pin_header_2.54mm_1x4; symbol RAMPS-FD-rescue:CONN_4 -> RAMPS-FD:1x4PinHeader; Fitted (none) -> yes; Ordering (none) -> LCSC: C124378; Price (USD) (none) -> 0,024235
- J9: renamed from P204; value X -> 1x4PinHeader; footprint rmc:CONN_KK_2.54_4W -> RAMPS-FD:pin_header_2.54mm_1x4; symbol RAMPS-FD-rescue:CONN_4 -> RAMPS-FD:1x4PinHeader; Fitted (none) -> yes; Ordering (none) -> LCSC: C124378; Price (USD) (none) -> 0,024235
- R10: renamed from R7; footprint Resistors_SMD:R_0603 -> RAMPS-FD:R_0603; symbol RAMPS-FD-rescue:R -> RAMPS-FD:10k; Fitted (none) -> yes; Ordering (none) -> LCSC: C238881; Price (USD) (none) -> 0,003395
- R11: renamed from R201; footprint Resistors_SMD:R_0603 -> RAMPS-FD:R_0603; symbol RAMPS-FD-rescue:R -> RAMPS-FD:100k; Fitted (none) -> yes; Ordering (none) -> LCSC: C237792; Price (USD) (none) -> 0,003527
- R6: renamed from R4; footprint Resistors_SMD:R_0603 -> RAMPS-FD:R_0603; symbol RAMPS-FD-rescue:R -> RAMPS-FD:10k; Fitted (none) -> yes; Ordering (none) -> LCSC: C238881; Price (USD) (none) -> 0,003395
- R7: renamed from R202; footprint Resistors_SMD:R_0603 -> RAMPS-FD:R_0603; symbol RAMPS-FD-rescue:R -> RAMPS-FD:100k; Fitted (none) -> yes; Ordering (none) -> LCSC: C237792; Price (USD) (none) -> 0,003527
- R8: renamed from R6; footprint Resistors_SMD:R_0603 -> RAMPS-FD:R_0603; symbol RAMPS-FD-rescue:R -> RAMPS-FD:10k; Fitted (none) -> yes; Ordering (none) -> LCSC: C238881; Price (USD) (none) -> 0,003395
- R9: renamed from R203; footprint Resistors_SMD:R_0603 -> RAMPS-FD:R_0603; symbol RAMPS-FD-rescue:R -> RAMPS-FD:100k; Fitted (none) -> yes; Ordering (none) -> LCSC: C237792; Price (USD) (none) -> 0,003527
- U3: renamed from U201; value X -> Pololu; footprint rmc:POLOLU -> RAMPS-FD:POLOLU; symbol RMC:POLOLU -> RAMPS-FD:Pololu; DriverReference (none) -> ?; Fitted (none) -> yes; Ordering (none) -> LCSC: 2x C27438; Price (USD) (none) -> 0,102
- U4: renamed from U202; value Y -> Pololu; footprint rmc:POLOLU -> RAMPS-FD:POLOLU; symbol RMC:POLOLU -> RAMPS-FD:Pololu; DriverReference (none) -> ?; Fitted (none) -> yes; Ordering (none) -> LCSC: 2x C27438; Price (USD) (none) -> 0,102
- U5: renamed from U203; value Z -> Pololu; footprint rmc:POLOLU -> RAMPS-FD:POLOLU; symbol RMC:POLOLU -> RAMPS-FD:Pololu; DriverReference (none) -> ?; Fitted (none) -> yes; Ordering (none) -> LCSC: 2x C27438; Price (USD) (none) -> 0,102
Connections:
- net labels added: +5V, UART1_RX_LV, UART1_TX_LV, UART_TMC, UART_TMC_1
- wire segments 135 -> 235
