File: RAMPS-FD/steppers2.sch (KiCad schematic (older format))
At the start: 15 parts, among them P207 3 2 1, P208 3 2 1, P209 3 2 1, P210 E2, P212 E1, P217 E0, U204 E2, U205 E1, U206 E0

Commit message: Inital Commit RAMPS FD v2.3. SPI Support for every Driver added.
Parts:
- removed P207, P208, P209: 3 2 1, Pin_Headers:Pin_Header_Straight_2x03_Pitch2.54mm, symbol CONN_3X2
- added P10, P11, P12: SPI Selector, Connector_PinHeader_2.54mm:PinHeader_2x04_P2.54mm_Vertical, symbol RAMPS-FD-rescue:CONN_4X2
- added P13, P14, P15: Pullup Sel., Connector_PinHeader_2.54mm:PinHeader_1x04_P2.54mm_Vertical, symbol RAMPS-FD-rescue:CONN_4
- added R10, R12, R14: 10k, Resistor_SMD:R_0603_1608Metric, symbol RAMPS-FD-rescue:R
- C204, C205, C206: symbol CP1 -> RAMPS-FD-rescue:CP1
- P210, P212, P217: symbol CONN_4 -> RAMPS-FD-rescue:CONN_4
- R207, R208, R210: symbol R -> RAMPS-FD-rescue:R
- U204, U205, U206: symbol POLOLU -> RMC:POLOLU
Connections:
- net labels added: D50-MISO, D51-MOSI, D52-SCK, STEP_E0_CS, STEP_E1_CS, STEP_E2_CS
- wire segments 94 -> 139
Other:
- note added: "Add jumpers for TMC2130 SPI"
- note added: "Use Jumpers to Connect the SPI Bus to your Stepperdrivers, \nfor example for TMC 2130, \nor to select the microstepping for your Pololu by connecting \nthe middle pin row to +V_Logic"
- moved on the sheet: R208, R210

Commit message: Added UART for Communication with TMC2209 Drivers, improved inverse-polarity protection, added Driver Protection. Two Layer Design
Parts:
- removed P10, P11, P12: SPI Selector, Connector_PinHeader_2.54mm:PinHeader_2x04_P2.54mm_Vertical, symbol RAMPS-FD-rescue:CONN_4X2
- removed P13, P14, P15: Pullup Sel., Connector_PinHeader_2.54mm:PinHeader_1x04_P2.54mm_Vertical, symbol RAMPS-FD-rescue:CONN_4
- added D14, D16, D18: DS110W, RAMPS-FD:D_SOD-123F, symbol RAMPS-FD:DS110W
- added D15, D17, D19: SMF36CA, RAMPS-FD:D_SOD-123F, symbol RAMPS-FD:SMF36CA
- added JP10, JP12, JP14: 4x3JumperArray, RAMPS-FD:4x3_2.54mm_Header, symbol RAMPS-FD:4x3JumperArray
- added JP11, JP13, JP15: 1x2JumperArray, RAMPS-FD:PinHeader_1x02_P2.54mm_Vertical, symbol RAMPS-FD:1x2JumperArray
- added R15: 1k, RAMPS-FD:R_0603, symbol RAMPS-FD:1k
- added VR20, VR21, VR22, VR23, VR24, VR25, VR26, VR27, VR28, VR29, VR30, VR31, VR32, VR33, VR34, VR35, VR36, VR37: 33V, RAMPS-FD:R_0603, symbol RAMPS-FD:33V
- C10: renamed from C205; value 100u 35V -> 100u_35V; footprint Capacitors_SMD:CP_Elec_6.3x7.7 -> RAMPS-FD:CP_Elec_6.3x7.7; symbol RAMPS-FD-rescue:CP1 -> RAMPS-FD:100u_35V; Fitted (none) -> yes; Ordering (none) -> LCSC: C88675; Price (USD) (none) -> 0,067122; Rating (none) -> #100uF #35V #20%
- C11: renamed from C204; value 100u 35V -> 100u_35V; footprint Capacitors_SMD:CP_Elec_6.3x7.7 -> RAMPS-FD:CP_Elec_6.3x7.7; symbol RAMPS-FD-rescue:CP1 -> RAMPS-FD:100u_35V; Fitted (none) -> yes; Ordering (none) -> LCSC: C88675; Price (USD) (none) -> 0,067122; Rating (none) -> #100uF #35V #20%
- C9: renamed from C206; value 100u 35V -> 100u_35V; footprint Capacitors_SMD:CP_Elec_6.3x7.7 -> RAMPS-FD:CP_Elec_6.3x7.7; symbol RAMPS-FD-rescue:CP1 -> RAMPS-FD:100u_35V; Fitted (none) -> yes; Ordering (none) -> LCSC: C88675; Price (USD) (none) -> 0,067122; Rating (none) -> #100uF #35V #20%
- J14: renamed from P217; value E0 -> 1x4PinHeader; footprint rmc:CONN_KK_2.54_4W -> RAMPS-FD:pin_header_2.54mm_1x4; symbol RAMPS-FD-rescue:CONN_4 -> RAMPS-FD:1x4PinHeader; Fitted (none) -> yes; Ordering (none) -> LCSC: C124378; Price (USD) (none) -> 0,024235
- J15: renamed from P212; value E1 -> 1x4PinHeader; footprint rmc:CONN_KK_2.54_4W -> RAMPS-FD:pin_header_2.54mm_1x4; symbol RAMPS-FD-rescue:CONN_4 -> RAMPS-FD:1x4PinHeader; Fitted (none) -> yes; Ordering (none) -> LCSC: C124378; Price (USD) (none) -> 0,024235
- J16: renamed from P210; value E2 -> 1x4PinHeader; footprint rmc:CONN_KK_2.54_4W -> RAMPS-FD:pin_header_2.54mm_1x4; symbol RAMPS-FD-rescue:CONN_4 -> RAMPS-FD:1x4PinHeader; Fitted (none) -> yes; Ordering (none) -> LCSC: C124378; Price (USD) (none) -> 0,024235
- R16: renamed from R14; footprint Resistor_SMD:R_0603_1608Metric -> RAMPS-FD:R_0603; symbol RAMPS-FD-rescue:R -> RAMPS-FD:10k; Fitted (none) -> yes; Ordering (none) -> LCSC: C238881; Price (USD) (none) -> 0,003395
- R17: renamed from R210; footprint Resistors_SMD:R_0603 -> RAMPS-FD:R_0603; symbol RAMPS-FD-rescue:R -> RAMPS-FD:100k; Fitted (none) -> yes; Ordering (none) -> LCSC: C237792; Price (USD) (none) -> 0,003527
- R18: renamed from R12; footprint Resistor_SMD:R_0603_1608Metric -> RAMPS-FD:R_0603; symbol RAMPS-FD-rescue:R -> RAMPS-FD:10k; Fitted (none) -> yes; Ordering (none) -> LCSC: C238881; Price (USD) (none) -> 0,003395
- R19: renamed from R208; footprint Resistors_SMD:R_0603 -> RAMPS-FD:R_0603; symbol RAMPS-FD-rescue:R -> RAMPS-FD:100k; Fitted (none) -> yes; Ordering (none) -> LCSC: C237792; Price (USD) (none) -> 0,003527
- R20: renamed from R10; footprint Resistor_SMD:R_0603_1608Metric -> RAMPS-FD:R_0603; symbol RAMPS-FD-rescue:R -> RAMPS-FD:10k; Fitted (none) -> yes; Ordering (none) -> LCSC: C238881; Price (USD) (none) -> 0,003395
- R21: renamed from R207; footprint Resistors_SMD:R_0603 -> RAMPS-FD:R_0603; symbol RAMPS-FD-rescue:R -> RAMPS-FD:100k; Fitted (none) -> yes; Ordering (none) -> LCSC: C237792; Price (USD) (none) -> 0,003527
- U7: renamed from U206; value E0 -> Pololu; footprint rmc:POLOLU -> RAMPS-FD:POLOLU; symbol RMC:POLOLU -> RAMPS-FD:Pololu; DriverReference (none) -> ?; Fitted (none) -> yes; Ordering (none) -> LCSC: 2x C27438; Price (USD) (none) -> 0,102
- U8: renamed from U205; value E1 -> Pololu; footprint rmc:POLOLU -> RAMPS-FD:POLOLU; symbol RMC:POLOLU -> RAMPS-FD:Pololu; DriverReference (none) -> ?; Fitted (none) -> yes; Ordering (none) -> LCSC: 2x C27438; Price (USD) (none) -> 0,102
- U9: renamed from U204; value E2 -> Pololu; footprint rmc:POLOLU -> RAMPS-FD:POLOLU; symbol RMC:POLOLU -> RAMPS-FD:Pololu; DriverReference (none) -> ?; Fitted (none) -> yes; Ordering (none) -> LCSC: 2x C27438; Price (USD) (none) -> 0,102
Connections:
- net labels added: +5V, UART2_RX_LV, UART2_TX_LV, UART_TMC, UART_TMC_1
- wire segments 139 -> 236
