File: RAMPS-FD/thermistor_inputs.sch (KiCad schematic (older format))
At the start: 14 parts, among them P301 THERMISTORS

Commit message: Inital Commit RAMPS FD v2.3. SPI Support for every Driver added.
Parts:
- C301, C302, C303, C501, C502, C503, C504, C505: symbol C -> RAMPS-FD-rescue:C
- L1: symbol INDUCTOR_SMALL -> RAMPS-FD-rescue:INDUCTOR_SMALL
- P301: symbol CONN_4X2 -> RAMPS-FD-rescue:CONN_4X2
- R301, R302, R303, R501: symbol R -> RAMPS-FD-rescue:R
Connections:
- wire segments 52 -> 71
Changed lines of the file:
@@
-EESchema Schematic File Version 2
-LIBS:RAMPS-FD-rescue
-LIBS:power
-LIBS:device
-LIBS:transistors
-LIBS:conn
-LIBS:linear
-LIBS:regul
-LIBS:74xx
-LIBS:cmos4000
-LIBS:adc-dac
-LIBS:memory
-LIBS:xilinx
-LIBS:microcontrollers
-LIBS:dsp
-LIBS:microchip
-LIBS:analog_switches
-LIBS:motorola
-LIBS:texas
-LIBS:intel
-LIBS:audio
-LIBS:interface
-LIBS:digital-audio
-LIBS:philips
-LIBS:display
-LIBS:cypress
-LIBS:siliconi
-LIBS:opto
-LIBS:atmel
-LIBS:contrib
-LIBS:valves
-LIBS:RMC
-LIBS:RAMPS-FD-cache
-EELAYER 25 0
+EESchema Schematic File Version 4
+EELAYER 30 0
 EELAYER END
 $Descr A4 11693 8268
@@
 Sheet 10 10
 Title "RAMPS-FD (RAMPS for Arduino Due)"
-Date "2016-07-17"
-Rev "v2.2"
+Date "2019-04-13"
+Rev "v2.3"
 Comp ""
-Comment1 "Derived from RAMPS 1.4 reprap.org/wiki/RAMPS1.4"
+Comment1 "Derived from RAMPS FD 2.2 by Bob Cousins github.com/bobc/bobc_hardware/"
 Comment2 "GPL v3"
-Comment3 "Bob Cousins 2016"
+Comment3 "Marius Krause 2019"
 Comment4 ""
 $EndDescr
 $Comp
-L C C504
+L RAMPS-FD-rescue:C C504
 U 1 1 519E9453
 P 5500 1800
@@
 $EndComp
 $Comp
-L C C505
+L RAMPS-FD-rescue:C C505
 U 1 1 519E9445
 P 5600 3600
@@
 $EndComp
 $Comp
-L C C503
+L RAMPS-FD-rescue:C C503
 U 1 1 519E9435
 P 5600 5100
@@
 From \nthermistors
 $Comp
-L C C502
+L RAMPS-FD-rescue:C C502
 U 1 1 517BAD21
 P 5650 6700
@@
 $EndComp
 $Comp
-L R R501
+L RAMPS-FD-rescue:R R501
 U 1 1 5178644E
 P 4000 6050
@@
 $EndComp
 $Comp
-L C C501
+L RAMPS-FD-rescue:C C501
 U 1 1 5178644D
 P 6100 6700
@@
 THERM3
 $Comp
-L CONN_4X2 P301
+L RAMPS-FD-rescue:CONN_4X2 P301
 U 1 1 517863D5
 P 2350 2550
@@
 THERM2
 $Comp
-L C C303
+L RAMPS-FD-rescue:C C303
 U 1 1 50FC3AB4
 P 6100 5100
@@
 $EndComp
 $Comp
-L R R303
+L RAMPS-FD-rescue:R R303
 U 1 1 50FC3AB3
 P 4000 4550
@@
 $EndComp
 $Comp
-L R R302
+L RAMPS-FD-rescue:R R302
 U 1 1 50FC3A9E
 P 4000 3050
@@
 $EndComp
 $Comp
-L C C302
+L RAMPS-FD-rescue:C C302
 U 1 1 50FC3A9D
 P 6100 3600
@@
 THERM0
 $Comp
-L C C301
+L RAMPS-FD-rescue:C C301
 U 1 1 50FC3A14
 P 6100 1800
@@
 $EndComp
 $Comp
-L R R301
+L RAMPS-FD-rescue:R R301
 U 1 1 50FC3A00
 P 3900 1250
@@
 $EndComp
 $Comp
-L GNDA #PWR0121
+L power:GNDA #PWR0121
 U 1 1 52CCBFF0
 P 1750 3000
@@
 $EndComp
 $Comp
-L +V_LOGIC #PWR0115
+L RMC:+V_LOGIC #PWR0115
 U 1 1 537E81B8
 P 1150 1025
@@
 $EndComp
 $Comp
-L INDUCTOR_SMALL L1
+L RAMPS-FD-rescue:INDUCTOR_SMALL L1
 U 1 1 5723B595
 P 1625 1175
@@
 	3250 2600 3250 4850
 Wire Wire Line
-	3250 4850 6500 4850
-Wire Wire Line
-	3100 1550 6450 1550
+	3250 4850 4000 4850
+Wire Wire Line
+	3100 1550 3900 1550
 Wire Wire Line
 	3100 1550 3100 2400
@@
 	5600 4850 5600 4950
 Wire Wire Line
-	3100 6400 6550 6400
+	3100 6400 4000 6400
 Wire Wire Line
 	3100 2700 3100 6400
@@
 Connection ~ 6100 7000
 Wire Wire Line
-	6100 6850 6100 7150
+	6100 6850 6100 7000
 Connection ~ 6100 6400
 Wire Wire Line
@@
 	3900 950  3900 1100
 Wire Wire Line
-	6100 1950 6100 2100
-Wire Wire Line
-	6100 3750 6100 3900
+	6100 1950 6100 2050
+Wire Wire Line
+	6100 3750 6100 3850
 Connection ~ 6100 3350
 Wire Wire Line
@@
 Connection ~ 6100 4850
 Wire Wire Line
-	6100 5250 6100 5400
+	6100 5250 6100 5350
 Wire Wire Line
 	1750 2600 1950 2600
@@
 	1950 2400 1750 2400
 Wire Wire Line
-	1750 2400 1750 3000
+	1750 2400 1750 2500
 Connection ~ 1750 2500
 Wire Wire Line
@@
 	3400 2500 3400 3350
 Wire Wire Line
-	3400 3350 6400 3350
+	3400 3350 4000 3350
 Wire Wire Line
 	6100 1650 6100 1550
@@
 	4000 2600 3775 2600
 $Comp
-L GNDA #PWR0116
+L power:GNDA #PWR0116
 U 1 1 5723EA8A
 P 6100 2100
@@
 $EndComp
 $Comp
-L GNDA #PWR0117
+L power:GNDA #PWR0117
 U 1 1 5723F10F
 P 6100 3900
@@
 $EndComp
 $Comp
-L GNDA #PWR0118
+L power:GNDA #PWR0118
 U 1 1 5723F49D
 P 6100 5400
@@
 $EndComp
 $Comp
-L GNDA #PWR0119
+L power:GNDA #PWR0119
 U 1 1 5723F505
 P 6100 7150
@@
 	1    0    0    -1
 $EndComp
+Wire Wire Line
+	5600 3350 6100 3350
+Wire Wire Line
+	6100 2050 6100 2100
+Wire Wire Line
+	6100 7000 6100 7150
+Wire Wire Line
+	6100 6400 6550 6400
+Wire Wire Line
+	1750 2600 1750 2700
+Wire Wire Line
+	6100 3350 6400 3350
+Wire Wire Line
+	6100 4850 6500 4850
+Wire Wire Line
+	1750 2700 1750 3000
+Wire Wire Line
+	1750 2500 1750 2600
+Wire Wire Line
+	5650 6400 6100 6400
+Wire Wire Line
+	6100 5350 6100 5400
+Wire Wire Line
+	5600 4850 6100 4850
+Wire Wire Line
+	5500 1550 6100 1550
+Wire Wire Line
+	6100 3850 6100 3900
+Wire Wire Line
+	6100 1550 6450 1550
+Wire Wire Line
+	3900 1550 5500 1550
+Wire Wire Line
+	4000 3350 5600 3350
+Wire Wire Line
+	4000 4850 5600 4850
+Wire Wire Line
+	4000 6400 5650 6400
 $EndSCHEMATC

Commit message: Added UART for Communication with TMC2209 Drivers, improved inverse-polarity protection, added Driver Protection. Two Layer Design
Parts:
- removed P301: THERMISTORS, Pin_Headers:Pin_Header_Straight_2x04_Pitch2.54mm, symbol RAMPS-FD-rescue:CONN_4X2
- added J32: 2x4PinHeader_2.54mm, RAMPS-FD:pin_header_2.54mm_2x4, symbol RAMPS-FD:2x4PinHeader_2.54mm
- C14: renamed from C504; footprint Capacitors_SMD:C_0603 -> RAMPS-FD:C_0603; symbol RAMPS-FD-rescue:C -> RAMPS-FD:100n; Fitted (none) -> yes; Ordering (none) -> LCSC: C85999; Price (USD) (none) -> 0,016915; Rating (none) -> #100nF #50V #5%
- C15: renamed from C301; footprint Capacitors_SMD:C_0603 -> RAMPS-FD:C_0603; symbol RAMPS-FD-rescue:C -> RAMPS-FD:10u; Fitted (none) -> yes; Ordering (none) -> LCSC: C96446; Price (USD) (none) -> 0,043979; Rating (none) -> #10uF #25V #10%
- C16: renamed from C505; footprint Capacitors_SMD:C_0603 -> RAMPS-FD:C_0603; symbol RAMPS-FD-rescue:C -> RAMPS-FD:100n; Fitted (none) -> yes; Ordering (none) -> LCSC: C85999; Price (USD) (none) -> 0,016915; Rating (none) -> #100nF #50V #5%
- C17: renamed from C302; footprint Capacitors_SMD:C_0603 -> RAMPS-FD:C_0603; symbol RAMPS-FD-rescue:C -> RAMPS-FD:10u; Fitted (none) -> yes; Ordering (none) -> LCSC: C96446; Price (USD) (none) -> 0,043979; Rating (none) -> #10uF #25V #10%
- C18: renamed from C503; footprint Capacitors_SMD:C_0603 -> RAMPS-FD:C_0603; symbol RAMPS-FD-rescue:C -> RAMPS-FD:100n; Fitted (none) -> yes; Ordering (none) -> LCSC: C85999; Price (USD) (none) -> 0,016915; Rating (none) -> #100nF #50V #5%
- C19: renamed from C303; footprint Capacitors_SMD:C_0603 -> RAMPS-FD:C_0603; symbol RAMPS-FD-rescue:C -> RAMPS-FD:10u; Fitted (none) -> yes; Ordering (none) -> LCSC: C96446; Price (USD) (none) -> 0,043979; Rating (none) -> #10uF #25V #10%
- C20: renamed from C502; footprint Capacitors_SMD:C_0603 -> RAMPS-FD:C_0603; symbol RAMPS-FD-rescue:C -> RAMPS-FD:100n; Fitted (none) -> yes; Ordering (none) -> LCSC: C85999; Price (USD) (none) -> 0,016915; Rating (none) -> #100nF #50V #5%
- C21: renamed from C501; footprint Capacitors_SMD:C_0603 -> RAMPS-FD:C_0603; symbol RAMPS-FD-rescue:C -> RAMPS-FD:10u; Fitted (none) -> yes; Ordering (none) -> LCSC: C96446; Price (USD) (none) -> 0,043979; Rating (none) -> #10uF #25V #10%
- FB2: renamed from L1; value FB -> FB0603; footprint Resistors_SMD:R_0603 -> RAMPS-FD:R_0603; symbol RAMPS-FD-rescue:INDUCTOR_SMALL -> RAMPS-FD:FB0603; Fitted (none) -> yes; Ordering (none) -> LCSC: C441755; Price (USD) (none) -> 0,032936; Rating (none) -> #500mA #390Ohm@100MHz
- R38: renamed from R301; footprint Resistors_SMD:R_0603 -> RAMPS-FD:R_0603; symbol RAMPS-FD-rescue:R -> RAMPS-FD:1k; Fitted (none) -> yes; Ordering (none) -> LCSC: C328340; Price (USD) (none) -> 0,003087
- R39: renamed from R302; footprint Resistors_SMD:R_0603 -> RAMPS-FD:R_0603; symbol RAMPS-FD-rescue:R -> RAMPS-FD:1k; Fitted (none) -> yes; Ordering (none) -> LCSC: C328340; Price (USD) (none) -> 0,003087
- R40: renamed from R303; footprint Resistors_SMD:R_0603 -> RAMPS-FD:R_0603; symbol RAMPS-FD-rescue:R -> RAMPS-FD:1k; Fitted (none) -> yes; Ordering (none) -> LCSC: C328340; Price (USD) (none) -> 0,003087
- R41: renamed from R501; footprint Resistors_SMD:R_0603 -> RAMPS-FD:R_0603; symbol RAMPS-FD-rescue:R -> RAMPS-FD:1k; Fitted (none) -> yes; Ordering (none) -> LCSC: C328340; Price (USD) (none) -> 0,003087
