File: RAMPS-FD/con_inputs.sch (KiCad schematic (older format))
At the start: 7 parts, among them P801 ENDSTOPS, P802 -X+ -Y+ -Z+, U801 74HC4050

Commit message: Inital Commit RAMPS FD v2.3. SPI Support for every Driver added.
Parts:
- C305: symbol C -> RAMPS-FD-rescue:C
- JP801: symbol JUMP_MINI -> RMC:JUMP_MINI
- P801: symbol CONN_6 -> RAMPS-FD-rescue:CONN_6
- P802: symbol CONN_6X2 -> RAMPS-FD-rescue:CONN_6X2
- RP801, RP802: symbol R_PACK4 -> RAMPS-FD-rescue:R_PACK4
- U801: symbol 4050_RMC -> RMC:4050_RMC
Changed lines of the file:
@@
-EESchema Schematic File Version 2
-LIBS:RAMPS-FD-rescue
-LIBS:power
-LIBS:device
-LIBS:transistors
-LIBS:conn
-LIBS:linear
-LIBS:regul
-LIBS:74xx
-LIBS:cmos4000
-LIBS:adc-dac
-LIBS:memory
-LIBS:xilinx
-LIBS:microcontrollers
-LIBS:dsp
-LIBS:microchip
-LIBS:analog_switches
-LIBS:motorola
-LIBS:texas
-LIBS:intel
-LIBS:audio
-LIBS:interface
-LIBS:digital-audio
-LIBS:philips
-LIBS:display
-LIBS:cypress
-LIBS:siliconi
-LIBS:opto
-LIBS:atmel
-LIBS:contrib
-LIBS:valves
-LIBS:RMC
-LIBS:RAMPS-FD-cache
-EELAYER 25 0
+EESchema Schematic File Version 4
+EELAYER 30 0
 EELAYER END
 $Descr A4 11693 8268
@@
 Sheet 8 10
 Title "RAMPS-FD (RAMPS for Arduino Due)"
-Date "2016-07-17"
-Rev "v2.2"
+Date "2019-04-13"
+Rev "v2.3"
 Comp ""
-Comment1 "Derived from RAMPS 1.4 reprap.org/wiki/RAMPS1.4"
+Comment1 "Derived from RAMPS FD 2.2 by Bob Cousins github.com/bobc/bobc_hardware/"
 Comment2 "GPL v3"
-Comment3 "Bob Cousins 2016"
+Comment3 "Marius Krause 2019"
 Comment4 ""
 $EndDescr
@@
 	1750 3750 3300 3750
 $Comp
-L +V_LOGIC #PWR0103
+L RMC:+V_LOGIC #PWR0103
 U 1 1 517866F1
 P 4250 2700
@@
 $EndComp
 $Comp
-L +V_LOGIC #PWR0104
+L RMC:+V_LOGIC #PWR0104
 U 1 1 517866E5
 P 4900 2200
@@
 $EndComp
 $Comp
-L GND #PWR0106
+L power:GND #PWR0106
 U 1 1 510D87E0
 P 4900 2800
@@
 $EndComp
 $Comp
-L C C305
+L RAMPS-FD-rescue:C C305
 U 1 1 510D87AD
 P 4900 2500
@@
 $EndComp
 $Comp
-L +5V #PWR0106
+L power:+5V #PWR0106
 U 1 1 50FF1A76
 P 800 1800
@@
 $EndComp
 $Comp
-L GND #PWR0108
+L power:GND #PWR0108
 U 1 1 50FF1A09
 P 4250 5100
@@
 X-MIN
 $Comp
-L GND #PWR0109
+L power:GND #PWR0109
 U 1 1 50FC388F
 P 700 4500
@@
 $EndComp
 $Comp
-L 4050_RMC U801
+L RMC:4050_RMC U801
 U 1 1 5244B8CC
 P 4450 3150
@@
 $EndComp
 $Comp
-L R_PACK4 RP801
+L RAMPS-FD-rescue:R_PACK4 RP801
 U 1 1 524E0304
 P 2550 2050
@@
 Connection ~ 2300 1650
 $Comp
-L R_PACK4 RP802
+L RAMPS-FD-rescue:R_PACK4 RP802
 U 1 1 524E0589
 P 3200 2050
@@
 NoConn ~ 2200 2250
 $Comp
-L +5V #PWR0109
+L power:+5V #PWR0109
 U 1 1 524E05B1
 P 2100 1100
@@
 $EndComp
 $Comp
-L JUMP_MINI JP801
+L RMC:JUMP_MINI JP801
 U 1 1 524E05B9
 P 2350 1350
@@
 Connection ~ 3050 1650
 $Comp
-L CONN_6X2 P802
+L RAMPS-FD-rescue:CONN_6X2 P802
 U 1 1 52B20629
 P 1350 3800
@@
 $EndComp
 $Comp
-L CONN_6 P801
+L RAMPS-FD-rescue:CONN_6 P801
 U 1 1 52B20647
 P 1350 2550

Commit message: Added UART for Communication with TMC2209 Drivers, improved inverse-polarity protection, added Driver Protection. Two Layer Design
Parts:
- removed P801: ENDSTOPS, Pin_Headers:Pin_Header_Straight_1x06_Pitch2.54mm, symbol RAMPS-FD-rescue:CONN_6
- removed P802: -X+ -Y+ -Z+, Pin_Headers:Pin_Header_Straight_2x06_Pitch2.54mm, symbol RAMPS-FD-rescue:CONN_6X2
- added J29: 3x6PinHeader, RAMPS-FD:6x3_2.54mm_Header, symbol RAMPS-FD:3x6PinHeader
- C13: renamed from C305; footprint Capacitors_SMD:C_0603 -> RAMPS-FD:C_0603; symbol RAMPS-FD-rescue:C -> RAMPS-FD:100n; Fitted (none) -> yes; Ordering (none) -> LCSC: C85999; Price (USD) (none) -> 0,016915; Rating (none) -> #100nF #50V #5%
- JP16: renamed from JP801; value PULLUPS -> 1x2JumperArray; footprint Pin_Headers:Pin_Header_Straight_1x02_Pitch2.54mm -> RAMPS-FD:PinHeader_1x02_P2.54mm_Vertical; symbol RMC:JUMP_MINI -> RAMPS-FD:1x2JumperArray; Fitted (none) -> yes; Ordering (none) -> LCSC: C124375; Price (USD) (none) -> 0,015147
- RP5: renamed from RP801; value 10k -> 10kArrayx4; footprint Resistors_SMD:R_Cat16-4 -> RAMPS-FD:R_Array_Convex_4x0603; symbol RAMPS-FD-rescue:R_PACK4 -> RAMPS-FD:10kArrayx4; Fitted (none) -> yes; Ordering (none) -> LCSC: C29718; Price (USD) (none) -> 0,007304
- RP6: renamed from RP802; value 10k -> 10kArrayx4; footprint Resistors_SMD:R_Cat16-4 -> RAMPS-FD:R_Array_Convex_4x0603; symbol RAMPS-FD-rescue:R_PACK4 -> RAMPS-FD:10kArrayx4; Fitted (none) -> yes; Ordering (none) -> LCSC: C29718; Price (USD) (none) -> 0,007304
- U11: renamed from U801; value 74HC4050 -> MC74LCX07; footprint Housings_SSOP:TSSOP-16_4.4x5mm_Pitch0.65mm -> RAMPS-FD:TSSOP-14_4.4x5mm_P0.65mm; symbol RMC:4050_RMC -> RAMPS-FD:MC74LCX07; Fitted (none) -> yes; Ordering (none) -> LCSC: C233625; Price (USD) (none) -> 0,171882
Connections:
- wire segments 61 -> 94

Commit message: Bug Notice for Enstop Header
Other:
- note added: "!BUG in V3!\nGND and Signal swaped at J29! \nAdapter needed"
Changed lines of the file:
@@
 Wire Wire Line
 	1750 2700 1900 2700
+Text Notes 1050 3450 0    60   ~ 0
+!BUG in V3!\nGND and Signal swaped at J29! \nAdapter needed
 $EndSCHEMATC
